File: Kicad-Files/Signals.kicad_sch (KiCad schematic)
At the start: 0 parts

Commit message: Created schematics for 1.1V circuit
Signed-off-by: Jakub Sobota <jakub.sobota@3mdeb.com>
Parts:
- added U2: TUSB7320, TUSB7320:Texas_tusb7340, symbol Interface_USB:TUSB7340

Commit message: Updated schematics for 1.1V circuit
Signed-off-by: Jakub Sobota <jakub.sobota@3mdeb.com>
Connections:
- net GND: now reaches U2.A53 (PAD)
- net GND: now also U2.B20 (GND)
Changed lines of the file:
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@@
 		(comment 2 "Jakub Sobota")
+	)
+	(junction
+		(at 86.36 158.75)
+		(diameter 0)
+		(color 0 0 0 0)
+	)
+	(wire
+		(pts
+			(xy 86.36 151.13) (xy 86.36 158.75)
+		)
+		(stroke
+			(width 0)
+			(type default)
+		)
+	)
+	(wire
+		(pts
+			(xy 88.9 151.13) (xy 88.9 158.75)
+		)
+		(stroke
+			(width 0)
+			(type default)
+		)
+	)
+	(wire
+		(pts
+			(xy 88.9 158.75) (xy 86.36 158.75)
+		)
+		(stroke
+			(width 0)
+			(type default)
+		)
+	)
+	(symbol
+		(lib_id "power:GND")
+		(at 86.36 158.75 0)
+		(unit 1)
+		(exclude_from_sim no)
+		(in_bom yes)
+		(on_board yes)
+		(dnp no)
+		(fields_autoplaced yes)
+		(property "Reference" "#PWR026"
+			(at 86.36 165.1 0)
+			(effects
+				(font
+					(size 1.27 1.27)
+				)
+				(hide yes)
+			)
+		)
+		(property "Value" "GND"
+			(at 86.36 163.83 0)
+			(effects
+				(font
+					(size 1.27 1.27)
+				)
+			)
+		)
+		(property "Footprint" ""
+			(at 86.36 158.75 0)
+			(effects
+				(font
+					(size 1.27 1.27)
+				)
+				(hide yes)
+			)
+		)
+		(property "Datasheet" ""
+			(at 86.36 158.75 0)
+			(effects
+				(font
+					(size 1.27 1.27)
+				)
+				(hide yes)
+			)
+		)
+		(property "Description" "Power symbol creates a global label with name \"GND\" , ground"
+			(at 86.36 158.75 0)
+			(effects
+				(font
+					(size 1.27 1.27)
+				)
+				(hide yes)
+			)
+		)
+		(pin "1"
+		)
+		(instances
+			(project ""
+				(path "/513f496d-ec7a-4c1e-814f-35a10c718f03/c66d1eec-955e-444d-af71-f46ce926b72b"
+					(reference "#PWR026")
+					(unit 1)
+				)
+			)
+		)
 	)
 	(symbol
@@
 		(pin "A21"
 		)
-		(pin "A8"
+		(pin "NC"
 		)
 		(pin "B21"

Commit message: Fixed signal integrity for USB data lines
Signed-off-by: Jakub Sobota <jakub.sobota@3mdeb.com>
Parts:
- added J2: USB_9PIN_Internal, Connectors:USB 9 Pin internal header, symbol Connectors:USB_9PIN_Internal
- U2: symbol Interface_USB:TUSB7340 -> TUSB7320:TUSB7320
Connections:
- net GND: now also J2.7 (GND), J2.8 (GND)
- net at U2.A13 (USB_DM_DN2): now also J2.3 (D-)
- net at U2.A20 (USB_DP_DN1): now also J2.6 (D+)
- net at U2.B12 (USB_DP_DN2): now also J2.5 (D+)
- net at U2.B18 (USB_DM_DN1): now also J2.4 (D-)
- new net +5V: J2.1 (5V), J2.2 (5V)
