File: Kicad-Files/untitled.kicad_sch (KiCad schematic)
At the start: 12 parts, among them U3 TPS74401

Commit message: Created 1.1V Circuit for USB Host IC
Signed-off-by: Jakub Sobota <jakub.sobota@3mdeb.com>
Parts:
- added F3: 1A, Fuse:Fuse_0603_1608Metric_Pad1.05x0.95mm_HandSolder, symbol Device:Fuse_Small
- C4, C7: footprint (none) -> Capacitor_SMD:C_0805_2012Metric_Pad1.18x1.45mm_HandSolder
- C5: value C_Small -> NOPOP; footprint (none) -> Capacitor_SMD:C_0402_1005Metric_Pad0.74x0.62mm_HandSolder
- C6, C8: footprint (none) -> Capacitor_SMD:C_0402_1005Metric_Pad0.74x0.62mm_HandSolder
- D5: footprint (none) -> Diode_SMD:D_0603_1608Metric_Pad1.05x0.95mm_HandSolder
- R5, R6, R7, R8, R9: footprint (none) -> Resistor_SMD:R_0402_1005Metric_Pad0.72x0.64mm_HandSolder
Connections:
- net +3.3V: now also F3.1; no longer C4.1, D5.2 (A), R8.1, U3.10 (BIAS), U3.5 (IN)
- new net: C4.1, D5.2 (A), F3.2, R8.1, U3.10 (BIAS), U3.5 (IN)
Changed lines of the file:
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@@
 	(title_block
 		(title "PCI2USB")
-		(date "2025-10-27")
+		(date "2025-10-29")
 		(rev "1.0.0")
 		(company "3mdeb Sp. z o.o")
@@
 	(wire
 		(pts
+			(xy 81.28 96.52) (xy 86.36 96.52)
+		)
+		(stroke
+			(width 0)
+			(type default)
+		)
+	)
+	(wire
+		(pts
 			(xy 142.24 83.82) (xy 142.24 85.09)
 		)
@@
 	(wire
 		(pts
-			(xy 81.28 96.52) (xy 86.36 96.52)
+			(xy 71.12 96.52) (xy 76.2 96.52)
 		)
 		(stroke
@@
 			)
 		)
-		(property "Footprint" ""
+		(property "Footprint" "Capacitor_SMD:C_0805_2012Metric_Pad1.18x1.45mm_HandSolder"
 			(at 160.02 100.33 0)
 			(effects
@@
 			)
 		)
-		(property "Datasheet" "~"
+		(property "Datasheet" "https://www.samsungsem.com/resources/file/global/support/product_catalog/MLCC.pdf"
 			(at 160.02 100.33 0)
 			(effects
@@
 			)
 		)
-		(property "Description" "Unpolarized capacitor, small symbol"
+		(property "Description" "X5R, 10%, 6.3V"
 			(at 160.02 100.33 0)
 			(effects
@@
 	(symbol
 		(lib_id "power:+3.3V")
-		(at 81.28 96.52 90)
+		(at 71.12 96.52 90)
 		(unit 1)
 		(exclude_from_sim no)
@@
 		(fields_autoplaced yes)
 		(property "Reference" "#PWR011"
-			(at 85.09 96.52 0)
+			(at 74.93 96.52 0)
 			(effects
 				(font
@@
 		)
 		(property "Value" "+3.3V"
-			(at 77.47 96.5199 90)
+			(at 67.31 96.5199 90)
 			(effects
 				(font
@@
 		)
 		(property "Footprint" ""
-			(at 81.28 96.52 0)
+			(at 71.12 96.52 0)
 			(effects
 				(font
@@
 		)
 		(property "Datasheet" ""
-			(at 81.28 96.52 0)
+			(at 71.12 96.52 0)
 			(effects
 				(font
@@
 		)
 		(property "Description" "Power symbol creates a global label with name \"+3.3V\""
-			(at 81.28 96.52 0)
+			(at 71.12 96.52 0)
 			(effects
 				(font
@@
 			)
 		)
-		(property "Footprint" ""
+		(property "Footprint" "Resistor_SMD:R_0402_1005Metric_Pad0.72x0.64mm_HandSolder"
 			(at 142.24 87.63 0)
 			(effects
@@
 			)
 		)
-		(property "Datasheet" "~"
+		(property "Datasheet" "https://industrial.panasonic.com/cdbs/www-data/pdf/RDA0000/AOA0000C304.pdf"
 			(at 142.24 87.63 0)
 			(effects
@@
 			)
 		)
-		(property "Description" "Resistor, small US symbol"
+		(property "Description" "1%, 100mW"
 			(at 142.24 87.63 0)
 			(effects
@@
 			)
 		)
-		(property "Footprint" ""
+		(property "Footprint" "Resistor_SMD:R_0402_1005Metric_Pad0.72x0.64mm_HandSolder"
 			(at 142.24 105.41 0)
 			(effects
@@
 			)
 		)
-		(property "Datasheet" "~"
+		(property "Datasheet" "https://industrial.panasonic.com/cdbs/www-data/pdf/RDA0000/AOA0000C304.pdf"
 			(at 142.24 105.41 0)
 			(effects
@@
 			)
 		)
-		(property "Description" "Resistor, small US symbol"
+		(property "Description" "0.05%, 62.5mW"
 			(at 142.24 105.41 0)
 			(effects
@@
 			)
 		)
-		(property "Footprint" ""
+		(property "Footprint" "Capacitor_SMD:C_0402_1005Metric_Pad0.74x0.62mm_HandSolder"
 			(at 110.49 82.55 0)
 			(effects
@@
 			)
 		)
-		(property "Datasheet" "~"
+		(property "Datasheet" "https://www.mouser.pl/datasheet/3/76/1/GRM155R70J104KA01-01A.pdf"
 			(at 110.49 82.55 0)
 			(effects
@@
 			)
 		)
-		(property "Description" "Unpolarized capacitor, small symbol"
+		(property "Description" "X7R, 10%, 6.3V"
 			(at 110.49 82.55 0)
 			(effects
@@
 			)
 		)
-		(property "Datasheet" ""
+		(property "Datasheet" "https://www.ti.com/lit/gpn/tps74401"
 			(at 128.27 83.82 0)
 			(effects
@@
 			)
 		)
-		(property "Footprint" ""
+		(property "Footprint" "Resistor_SMD:R_0402_1005Metric_Pad0.72x0.64mm_HandSolder"
 			(at 142.24 99.06 0)
 			(effects
@@
 			)
 		)
-		(property "Datasheet" "~"
+		(property "Datasheet" "https://industrial.panasonic.com/cdbs/www-data/pdf/RDA0000/AOA0000C304.pdf"
 			(at 142.24 99.06 0)
 			(effects
@@
 			)
 		)
-		(property "Description" "Resistor, small US symbol"
+		(property "Description" "1%, 100mW"
 			(at 142.24 99.06 0)
 			(effects
@@
 			)
 		)
-		(property "Footprint" ""
+		(property "Footprint" "Diode_SMD:D_0603_1608Metric_Pad1.05x0.95mm_HandSolder"
 			(at 86.36 100.33 0)
 			(effects
@@
 			)
 		)
-		(property "Datasheet" "~"
+		(property "Datasheet" "https://www.mouser.pl/datasheet/3/308/1/APHD1608LCGCK.pdf"
 			(at 86.36 100.33 0)
 			(effects
@@
 			)
 		)
-		(property "Description" "Light emitting diode"
+		(property "Description" "GREEN Light emitting diode"
 			(at 86.36 100.33 0)
 			(effects
@@
 		(on_board yes)
 		(dnp no)
-		(fields_autoplaced yes)
 		(property "Reference" "C5"
-			(at 118.11 104.1462 0)
-			(effects
-				(font
-					(size 1.27 1.27)
-				)
-				(justify left)
-			)
-		)
-		(property "Value" "C_Small"
-			(at 118.11 106.6862 0)
-			(effects
-				(font
-					(size 1.27 1.27)
-				)
-				(justify left)
-				(hide yes)
-			)
-		)
-		(property "Footprint" ""
+			(at 117.348 104.394 0)
+			(effects
+				(font
+					(size 1.27 1.27)
+				)
+				(justify left)
+			)
+		)
+		(property "Value" "NOPOP"
+			(at 117.602 106.68 0)
+			(effects
+				(font
+					(size 1.27 1.27)
+				)
+				(justify left)
+			)
+		)
+		(property "Footprint" "Capacitor_SMD:C_0402_1005Metric_Pad0.74x0.62mm_HandSolder"
 			(at 115.57 105.41 0)
 			(effects
@@
 			)
 		)
-		(property "Description" "Unpolarized capacitor, small symbol"
+		(property "Description" "NOPOP"
 			(at 115.57 105.41 0)
 			(effects
@@
 			)
 		)
-		(property "Footprint" ""
+		(property "Footprint" "Resistor_SMD:R_0402_1005Metric_Pad0.72x0.64mm_HandSolder"
 			(at 86.36 109.22 0)
 			(effects
@@
 			)
 		)
-		(property "Datasheet" "~"
+		(property "Datasheet" "https://www.vishay.com/docs/20035/dcrcwe3.pdf"
 			(at 86.36 109.22 0)
 			(effects
@@
 			)
 		)
-		(property "Description" "Resistor, small US symbol"
+		(property "Description" "1%, 63mW"
 			(at 86.36 109.22 0)
 			(effects
@@
 			)
 		)
-		(property "Footprint" ""
+		(property "Footprint" "Resistor_SMD:R_0402_1005Metric_Pad0.72x0.64mm_HandSolder"
 			(at 106.68 92.71 0)
 			(effects
@@
 			)
 		)
-		(property "Datasheet" "~"
+		(property "Datasheet" "https://industrial.panasonic.com/cdbs/www-data/pdf/RDA0000/AOA0000C304.pdf"
 			(at 106.68 92.71 0)
 			(effects
@@
 			)
 		)
-		(property "Description" "Resistor, small US symbol"
+		(property "Description" "1%, 100mW"
 			(at 106.68 92.71 0)
 			(effects
@@
 	)
 	(symbol
+		(lib_id "Device:Fuse_Small")
+		(at 78.74 96.52 0)
+		(unit 1)
+		(exclude_from_sim no)
+		(in_bom yes)
+		(on_board yes)
+		(dnp no)
+		(fields_autoplaced yes)
+		(property "Reference" "F3"
+			(at 78.74 91.44 0)
+			(effects
+				(font
+					(size 1.27 1.27)
+				)
+			)
+		)
+		(property "Value" "1A"
+			(at 78.74 93.98 0)
+			(effects
+				(font
+					(size 1.27 1.27)
+				)
+			)
+		)
+		(property "Footprint" "Fuse:Fuse_0603_1608Metric_Pad1.05x0.95mm_HandSolder"
+			(at 78.74 96.52 0)
+			(effects
+				(font
+					(size 1.27 1.27)
+				)
+				(hide yes)
+			)
+		)
+		(property "Datasheet" "https://www.vishay.com/doc?28747"
+			(at 78.74 96.52 0)
+			(effects
+				(font
+					(size 1.27 1.27)
+				)
+				(hide yes)
+			)
+		)
+		(property "Description" "Fast Act Fuse"
+			(at 78.74 96.52 0)
+			(effects
+				(font
+					(size 1.27 1.27)
+				)
+				(hide yes)
+			)
+		)
+		(pin "2"
+		)
+		(pin "1"
+		)
+		(instances
+			(project "PCI2USB"
+				(path "/513f496d-ec7a-4c1e-814f-35a10c718f03/641a18fa-9239-44e7-9711-1a374441a862"
+					(reference "F3")
+					(unit 1)
+				)
+			)
+		)
+	)
+	(symbol
 		(lib_id "power:GND")
 		(at 97.79 105.41 0)
@@
 			)
 		)
-		(property "Footprint" ""
+		(property "Footprint" "Capacitor_SMD:C_0805_2012Metric_Pad1.18x1.45mm_HandSolder"
 			(at 97.79 99.06 0)
 			(effects
@@
 			)
 		)
-		(property "Datasheet" "~"
+		(property "Datasheet" "https://search.murata.co.jp/Ceramy/image/img/A01X/G101/ENG/GRM21BR70J106KA73-01A.pdf"
 			(at 97.79 99.06 0)
 			(effects
@@
 			)
 		)
-		(property "Description" "Unpolarized capacitor, small symbol"
+		(property "Description" "X7R, 10%, 6.3V"
 			(at 97.79 99.06 0)
 			(effects
@@
 			)
 		)
-		(property "Footprint" ""
+		(property "Footprint" "Capacitor_SMD:C_0402_1005Metric_Pad0.74x0.62mm_HandSolder"
 			(at 157.48 88.9 0)
 			(effects
@@
 			)
 		)
-		(property "Datasheet" "~"
+		(property "Datasheet" "https://www.mouser.pl/datasheet/3/76/1/GRM155R70J104KA01-01A.pdf"
 			(at 157.48 88.9 0)
 			(effects
@@
 			)
 		)
-		(property "Description" "Unpolarized capacitor, small symbol"
+		(property "Description" "X7R, 10%, 6.3V"
 			(at 157.48 88.9 0)
 			(effects

Commit message: Updated schematics for 1.1V circuit
Signed-off-by: Jakub Sobota <jakub.sobota@3mdeb.com>
Parts:
- D5: footprint Diode_SMD:D_0603_1608Metric_Pad1.05x0.95mm_HandSolder -> LED_SMD:LED_0603_1608Metric_Pad1.05x0.95mm_HandSolder
Connections:
- net +1.1V: now also U3.18 (OUT), U3.19 (OUT), U3.20 (OUT)
- net +3.3V: no longer R7.1
- net GND: now also U3.13 (NC), U3.14 (NC), U3.17 (NC), U3.21 (PAD), U3.3 (NC), U3.4 (NC)
- net at C4.1, D5.2 (A), F3.2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: now also R7.1, U3.6 (IN), U3.7 (IN), U3.8 (IN)
Other:
- moved on the sheet: C4, C5, C6, C7, C8, D5, F3, R5, R6, R7, R8, R9

Commit message: Fixed signal integrity for USB data lines
Signed-off-by: Jakub Sobota <jakub.sobota@3mdeb.com>
Parts:
- removed U3: TPS74401, Package_DFN_QFN:Texas_RGW0020A_VQFN-20-1EP_5x5mm_P0.65mm_EP3.15x3.15mm_ThermalVias, symbol Regulator_Linear:TPS74401_VQFN
- added U3: TPS74401, Package_DFN_QFN:Texas_RGW0020A_VQFN-20-1EP_5x5mm_P0.65mm_EP3.15x3.15mm_ThermalVias, symbol DC-DC Converter:TPS74401_VQFN
Connections:
- net +1.1V: now also U3.1 (OUT), U3.18 (OUT), U3.19 (OUT), U3.20 (OUT)
- net GND: now also U3.12 (GND), U3.13 (NC), U3.14 (NC), U3.17 (NC), U3.21 (PAD), U3.3 (NC), U3.4 (NC)
- net GRSTZ: now also U3.9 (PG)
- net at C4.1, D5.2 (A), F3.2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: now also U3.10 (BIAS), U3.5 (IN), U3.6 (IN), U3.7 (IN), U3.8 (IN)
- net at R5.2, R6.2: now also U3.16 (FB)
- net at C8.2, R8.2: now also U3.11 (EN)
- net at C5.1: now also U3.15 (SS)
Changed lines of the file:
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@@
+	)
+	(symbol
+		(lib_id "DC-DC Converter:TPS74401_VQFN")
+		(at 133.35 93.98 0)
+		(unit 1)
+		(exclude_from_sim no)
+		(in_bom yes)
+		(on_board yes)
+		(dnp no)
+		(fields_autoplaced yes)
+		(property "Reference" "U3"
+			(at 139.065 77.47 0)
+			(effects
+				(font
+					(size 1.27 1.27)
+				)
+			)
+		)
+		(property "Value" "TPS74401"
+			(at 139.065 80.01 0)
+			(effects
+				(font
+					(size 1.27 1.27)
+				)
+			)
+		)
+		(property "Footprint" "Package_DFN_QFN:Texas_RGW0020A_VQFN-20-1EP_5x5mm_P0.65mm_EP3.15x3.15mm_ThermalVias"
+			(at 153.67 109.22 0)
+			(effects
+				(font
+					(size 1.27 1.27)
+				)
+				(hide yes)
+			)
+		)
+		(property "Datasheet" "https://www.ti.com/lit/gpn/tps74401"
+			(at 138.43 74.93 0)
+			(effects
+				(font
+					(size 1.27 1.27)
+				)
+				(hide yes)
+			)
+		)
+		(property "Description" "0.8 to 3.6V adjustable, 3.0-A, Ultra-LDO with Programmable Soft-Start"
+			(at 149.606 114.808 0)
+			(effects
+				(font
+					(size 1.27 1.27)
+				)
+				(hide yes)
+			)
+		)
+		(pin "9"
+		)
+		(pin "17"
+		)
+		(pin "18"
+		)
+		(pin "10"
+		)
+		(pin "12"
+		)
+		(pin "7"
+		)
+		(pin "14"
+		)
+		(pin "16"
+		)
+		(pin "19"
+		)
+		(pin "15"
+		)
+		(pin "1"
+		)
+		(pin "8"
+		)
+		(pin "21"
+		)
+		(pin "11"
+		)
+		(pin "3"
+		)
+		(pin "6"
+		)
+		(pin "20"
+		)
+		(pin "2"
+		)
+		(pin "4"
+		)
+		(pin "13"
+		)
+		(pin "5"
+		)
+		(instances
+			(project ""
+				(path "/513f496d-ec7a-4c1e-814f-35a10c718f03/641a18fa-9239-44e7-9711-1a374441a862"
+					(reference "U3")
+					(unit 1)
+				)
+			)
+		)
 	)
 	(symbol
@@
 					(unit 1)
 				)
-			)
-		)
-	)
-	(symbol
-		(lib_id "Regulator_Linear:TPS74401_VQFN")
-		(at 133.35 93.98 0)
-		(unit 1)
-		(exclude_from_sim no)
-		(in_bom yes)
-		(on_board yes)
-		(dnp no)
-		(fields_autoplaced yes)
-		(property "Reference" "U3"
-			(at 138.43 78.74 0)
-			(effects
-				(font
-					(size 1.27 1.27)
-				)
-			)
-		)
-		(property "Value" "TPS74401"
-			(at 138.43 81.28 0)
-			(effects
-				(font
-					(size 1.27 1.27)
-				)
-			)
-		)
-		(property "Footprint" "Package_DFN_QFN:Texas_RGW0020A_VQFN-20-1EP_5x5mm_P0.65mm_EP3.15x3.15mm_ThermalVias"
-			(at 153.67 109.22 0)
-			(effects
-				(font
-					(size 1.27 1.27)
-				)
-				(hide yes)
-			)
-		)
-		(property "Datasheet" "https://www.ti.com/lit/gpn/tps74401"
-			(at 138.43 78.74 0)
-			(effects
-				(font
-					(size 1.27 1.27)
-				)
-				(hide yes)
-			)
-		)
-		(property "Description" "0.8 to 3.6V adjustable, 3.0-A, Ultra-LDO with Programmable Soft-Start"
-			(at 149.606 114.808 0)
-			(effects
-				(font
-					(size 1.27 1.27)
-				)
-				(hide yes)
-			)
-		)
-		(pin "16"
-		)
-		(pin "18"
-		)
-		(pin "9"
-		)
-		(pin "13"
-		)
-		(pin "20"
-		)
-		(pin "4"
-		)
-		(pin "3"
-		)
-		(pin "5"
-		)
-		(pin "12"
-		)
-		(pin "2"
-		)
-		(pin "14"
-		)
-		(pin "19"
-		)
-		(pin "15"
-		)
-		(pin "10"
-		)
-		(pin "11"
-		)
-		(pin "8"
-		)
-		(pin "7"
-		)
-		(pin "17"
-		)
-		(pin "6"
-		)
-		(pin "1"
-		)
-		(pin "21"
-		)
-		(instances
-			(project ""
-				(path "/513f496d-ec7a-4c1e-814f-35a10c718f03/641a18fa-9239-44e7-9711-1a374441a862"
-					(reference "U3")
-					(unit 1)
-				)
