File: Kicad-Files/PCI2USB.kicad_pcb (KiCad board)
At the start: 4 copper layers, 22 x 80 mm, 17 parts, among them U1 TPS61023

Commit message: Updated schematics and board layout
Signed-off-by: Jakub Sobota <jakub.sobota@3mdeb.com>
Parts:
- added J2: USB 9 Pin Connecetor, Connectors:USB 9 Pin internal header, F.Cu at (146.1, 96.0)
- REF IC: moved to B.Cu
- moved F2 7.49 mm to (139.2, 101.5)
- moved C1 7.23 mm to (140.5, 117.1)
- moved D1 7.23 mm to (137.4, 120.5)
- moved F1 7.23 mm to (139.1, 122.3)
- moved L1 7.23 mm to (144.5, 113.4)
- moved R4 7.23 mm to (141.2, 104.2)
- moved C2 7.23 mm to (139.5, 109.1)
- moved C3 7.23 mm to (139.5, 106.8)
- moved D3 7.23 mm to (139.9, 120.2)
- moved D4 7.23 mm to (139.1, 103.1)
- moved R1 7.23 mm to (137.4, 114.5)
- moved R2 7.23 mm to (137.4, 116.1)
- moved R3 7.23 mm to (137.1, 119.4)
- moved U1 7.23 mm to (140.3, 113.5)
- moved D2 7.23 mm to (139.6, 104.9)
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Connections:
- U$1 pad P$29: (no net) -> PERn1
- U$1 pad P$31: (no net) -> PERp1
- U$1 pad P$35: (no net) -> PETn1
- U$1 pad P$37: (no net) -> PETp1
- U$1 pad P$38: (no net) -> DEVSLP
- U$1 pad P$47: (no net) -> PETn0
- U$1 pad P$49: (no net) -> PETp0
- U$1 pad P$50: (no net) -> PERST
- U$1 pad P$52: (no net) -> CLKREQ
- U$1 pad P$54: (no net) -> PEWAKE
Routing:
- net GND: track 214.6 -> 73.3 mm, vias 53 -> 51
- net +3.3V: track 39.4 -> 22.4 mm, vias 6 -> 5
- net +5V: track 0.00 -> 12.7 mm, vias 0 -> 4
- net PETn1: track 0.00 -> 5.79 mm, vias 0 -> 1
- net PERn1: track 0.00 -> 5.79 mm, vias 0 -> 1
- net PERp1: track 0.00 -> 4.73 mm, vias 0 -> 1
- net PETp1: track 0.00 -> 4.53 mm, vias 0 -> 1

Commit message: Fixed DRC Warnings and Errors
Signed-off-by: Jakub Sobota <jakub.sobota@3mdeb.com>
Parts:
- REF IC: moved to F.Cu
- moved REF IC 3.66 mm to (150.8, 119.6), turned to 180 degrees
- moved L1 2.81 mm to (145.2, 110.7)
- moved D1 0.11 mm to (137.4, 120.6)
- moved R4 0.10 mm to (141.3, 104.2)
- moved D3 0.06 mm to (139.8, 120.2)
Connections:
- U$1 pad NC: NC -> (no net)
Routing:
- net GND: track 73.3 -> 64.1 mm, vias 51 -> 50
- net PETn1: track 5.79 -> 0.00 mm, vias 1 -> 0
- net PERn1: track 5.79 -> 0.00 mm, vias 1 -> 0
- net PETp1: track 4.53 -> 0.00 mm, vias 1 -> 0
- net PERp1: track 4.73 -> 0.21 mm, vias 1 -> 0
- net Net-(U1-SW): track 5.60 -> 8.79 mm

Commit message: Created schematics for 1.1V circuit
Signed-off-by: Jakub Sobota <jakub.sobota@3mdeb.com>
Parts:
- C2, C3: value 22 μF -> 33 μF; footprint Capacitor_SMD:C_1206_3216Metric_Pad1.33x1.80mm_HandSolder -> Capacitor_SMD:C_0805_2012Metric_Pad1.18x1.45mm_HandSolder
- R3, R4: footprint Resistor_SMD:R_0201_0603Metric_Pad0.64x0.40mm_HandSolder -> Resistor_SMD:R_0402_1005Metric_Pad0.72x0.64mm_HandSolder
- moved R4 0.21 mm to (141.5, 104.3)
- moved D2 0.16 mm to (139.4, 104.9)
- moved D1 0.15 mm to (137.3, 120.7)
- moved R3 0.15 mm to (137.2, 119.2)
Connections:
- REF IC pad A53: (no net) -> GND
- U$1 pad P$2: +3.3V -> +3.3V_CHIP
Routing:
- net GND: track 64.1 -> 90.8 mm, vias 50 -> 61
- net +3.3V: track 22.3 -> 17.9 mm, vias 5 -> 4
- net +3.3V_CHIP: track 0.00 -> 4.21 mm, vias 0 -> 1

Commit message: Created 1.1V Circuit for USB Host IC
Signed-off-by: Jakub Sobota <jakub.sobota@3mdeb.com>
Parts:
- removed REF IC: Texas_WQFN-MR-100_3x3-DapStencil, Package_DFN_QFN:Texas_WQFN-MR-100_3x3-DapStencil
- added C4: 10 μF, Capacitor_SMD:C_0805_2012Metric_Pad1.18x1.45mm_HandSolder, B.Cu at (148.3, 122.4)
- added C5: NOPOP, Capacitor_SMD:C_0402_1005Metric_Pad0.74x0.62mm_HandSolder, B.Cu at (140.5, 120.4)
- added C6: 0.1 μF, Capacitor_SMD:C_0402_1005Metric_Pad0.74x0.62mm_HandSolder, B.Cu at (137.2, 121.1)
- added C7: 22 μF, Capacitor_SMD:C_0805_2012Metric_Pad1.18x1.45mm_HandSolder, B.Cu at (143.5, 116.2)
- added C8: 0.01 μF, Capacitor_SMD:C_0402_1005Metric_Pad0.74x0.62mm_HandSolder, B.Cu at (138.9, 121.6)
- added D5: LED, LED_SMD:LED_0603_1608Metric_Pad1.05x0.95mm_HandSolder, F.Cu at (142.0, 123.4)
- added F3: 1A, Fuse:Fuse_0603_1608Metric_Pad1.05x0.95mm_HandSolder, B.Cu at (151.8, 124.3)
- added R5: 4.99 KOhm, Resistor_SMD:R_0402_1005Metric_Pad0.72x0.64mm_HandSolder, B.Cu at (141.4, 117.7)
- added R6: 1.87 KOhm, Resistor_SMD:R_0402_1005Metric_Pad0.72x0.64mm_HandSolder, B.Cu at (143.7, 117.7)
- added R7: 10 KOhm, Resistor_SMD:R_0402_1005Metric_Pad0.72x0.64mm_HandSolder, B.Cu at (137.2, 122.2)
- added R8: 4.7 KOhm, Resistor_SMD:R_0402_1005Metric_Pad0.72x0.64mm_HandSolder, B.Cu at (139.9, 122.6)
- added R9: 330 Ohm, Resistor_SMD:R_0402_1005Metric_Pad0.72x0.64mm_HandSolder, F.Cu at (144.2, 123.2)
- added U2: TUSB7320, TUSB7320:Texas_tusb7340, F.Cu at (151.2, 119.0)
- added U3: TPS74401, Package_DFN_QFN:Texas_RGW0020A_VQFN-20-1EP_5x5mm_P0.65mm_EP3.15x3.15mm_ThermalVias, B.Cu at (144.1, 121.4)
- C2, C3: value 33 μF -> 22 μF
- F1: value 4A -> 5A
Connections:
- J2 pad 9: (no net) -> unconnected-(J2-Pin_9-Pad9)
Routing:
- net GND: track 90.8 -> 34.7 mm, vias 61 -> 53
- net GRSTZ: track 0.00 -> 9.15 mm, vias 0 -> 2
- net Net-(D5-A): track 0.00 -> 5.85 mm, vias 0 -> 1
- net +3.3V_CHIP: track 4.21 -> 5.78 mm
- net Net-(U3-FB): track 0.00 -> 1.09 mm
- added copper zone on B.Cu, net GND

Commit message: Created 1.1V Circuit for USB Host IC
Signed-off-by: Jakub Sobota <jakub.sobota@3mdeb.com>
Routing:
- net Net-(D5-A): track 5.85 -> 0.53 mm
- added copper zone on B.Cu, net Net-(D5-A)
Changed lines of the file:
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@@
-	(gr_poly
-		(pts
-			(xy 143.849773 124.944) (xy 151.181 124.944) (xy 151.465 124.66) (xy 151.465 123.265) (xy 150.71 122.51)
-			(xy 145.94 122.52) (xy 145.94 123.04) (xy 145.676 123.24) (xy 143.860198 123.24)
-		)
-		(stroke
-			(width 0)
-			(type solid)
-		)
-		(fill yes)
-		(layer "B.Cu")
-		(net 29)
-	)
 	(gr_poly
 		(pts
@@
 	(gr_poly
 		(pts
-			(xy 148.87 122.23) (xy 146.4625 122.23) (xy 146.4625 120.56) (xy 148.04 120.56) (xy 148.74 119.86)
-			(xy 149.99 121.11)
-		)
-		(stroke
-			(width 0)
-			(type solid)
-		)
-		(fill yes)
-		(layer "B.Cu")
-		(net 1)
-	)
-	(gr_poly
-		(pts
 			(xy 142.725202 119.44) (xy 142.44 119.18) (xy 141.72 118.51) (xy 141.71 118.02) (xy 141.714369 117.49)
 			(xy 143.329821 117.49) (xy 143.327499 118.10397) (xy 142.88 118.502553) (xy 142.88 119.44)
@@
 		(layer "B.Cu")
 		(net 36)
-	)
-	(gr_poly
-		(pts
-			(xy 142.97 123.339573) (xy 142.97 124.847738) (xy 140.720578 124.857271) (xy 140.727082 124.375963)
-			(xy 141.01 124.122061) (xy 141.01 123.65) (xy 140.810914 123.46343) (xy 138.415935 123.453281) (xy 137.566787 122.678331)
-			(xy 137.556666 121.98) (xy 138.079996 121.98) (xy 138.103524 122.497529) (xy 138.635898 122.938858)
-			(xy 140.557844 122.92818) (xy 141.267224 123.330515)
-		)
-		(stroke
-			(width 0.2)
-			(type solid)
-		)
-		(fill yes)
-		(layer "B.Cu")
-		(net 29)
-	)
-	(gr_poly
-		(pts
-			(xy 140.25 121.337429) (xy 140.25 120.669046) (xy 137.5 120.669046) (xy 137.5 121.337429)
-		)
-		(stroke
-			(width 0.2)
-			(type solid)
-		)
-		(fill yes)
-		(layer "B.Cu")
-		(net 1)
-	)
-	(gr_poly
-		(pts
-			(xy 145.1 122.39) (xy 145.27 122.22) (xy 146.99 122.23) (xy 146.99 121.38) (xy 146.99 120.55) (xy 145.26 120.55)
-			(xy 145.1 120.39) (xy 145.1 121.39)
-		)
-		(stroke
-			(width 0)
-			(type solid)
-		)
-		(fill yes)
-		(layer "B.Cu")
-		(net 1)
 	)
 	(gr_line
@@
 	)
 	(segment
-		(start 142.806 124.846)
-		(end 146.538386 124.846)
-		(width 0.2)
-		(layer "B.Cu")
-		(net 29)
-	)
-	(segment
-		(start 146.538386 124.846)
-		(end 147.657386 123.727)
-		(width 0.2)
-		(layer "B.Cu")
-		(net 29)
-	)
-	(segment
 		(start 137.7875 122.1775)
 		(end 137.82 122.21)
@@
 	)
 	(zone
-		(net 1)
-		(net_name "GND")
+		(net 29)
+		(net_name "Net-(D5-A)")
 		(locked yes)
 		(layer "B.Cu")
-		(hatch edge 0.5)
-		(priority 1)
-		(connect_pads
+		(hatch full 0.25)
+		(priority 2)
+		(connect_pads yes
 			(clearance 0.2)
 		)
-		(min_thickness 0.25)
+		(min_thickness 0.22)
 		(filled_areas_thickness no)
 		(fill yes
 			(thermal_gap 0.2)
 			(thermal_bridge_width 0.25)
+			(smoothing chamfer)
+			(radius 0.2)
+		)
+		(polygon
+			(pts
+				(xy 151.483637 124.94) (xy 151.199637 125.224) (xy 140.638637 125.24) (xy 140.618637 124.09) (xy 137.8 123.75)
+				(xy 136.72 122.64) (xy 136.888637 121.86) (xy 138.498637 121.85) (xy 139.988637 122.59) (xy 141.92 123.18)
+				(xy 142.75 123.17) (xy 145.43 123.17) (xy 145.378637 122.39) (xy 151.428637 122.39)
+			)
+		)
+	)
+	(zone
+		(net 1)
+		(net_name "GND")
+		(locked yes)
+		(layer "B.Cu")
+		(hatch edge 0.5)
+		(priority 1)
+		(connect_pads yes
+			(clearance 0.2)
+		)
+		(min_thickness 0.2)
+		(filled_areas_thickness no)
+		(fill yes
+			(thermal_gap 0.2)
+			(thermal_bridge_width 0.3)
 			(smoothing fillet)
-			(radius 1.2)
+			(radius 0.2)
+			(island_removal_mode 1)
+			(island_area_min 10)
 		)
 		(polygon

Commit message: Updated schematics for 1.1V circuit
Signed-off-by: Jakub Sobota <jakub.sobota@3mdeb.com>
Connections:
- F3 pad 1: +3.3V_CHIP -> +3.3V
- U$1 pad P$2: +3.3V_CHIP -> +3.3V
- U2 pad B20: unconnected-(U2-VSS-PadB20) -> GND
- U2 pad NC: (no net) -> unconnected-(U2-USB_SSTXN_DN4-PadNC)_11
- U3 pad 2: GND -> unconnected-(U3-NC-Pad2)
Routing:
- net +3.3V: track 17.9 -> 0.52 mm, vias 4 -> 5
- net +3.3V_CHIP: track 5.78 -> 0.00 mm, vias 1 -> 0
- net GND: track 34.7 -> 38.3 mm
- net Net-(U3-FB): track 1.09 -> 0.01 mm
- net +1.1V: vias 0 -> 1
- added copper zone on B.Cu, net +3.3V

Commit message: Fixed signal integrity for USB data lines
Signed-off-by: Jakub Sobota <jakub.sobota@3mdeb.com>
Parts:
- J2: value USB 9 Pin Connecetor -> USB_9PIN_Internal
- moved J2 0.95 mm to (146.1, 95.0)
Connections:
- J2 pad 3: unconnected-(J2-Pin_3-Pad3) -> Net-(U2-USB_DM_DN2)
- J2 pad 4: unconnected-(J2-Pin_4-Pad4) -> Net-(U2-USB_DM_DN1)
- J2 pad 5: unconnected-(J2-Pin_5-Pad5) -> Net-(U2-USB_DP_DN2)
- J2 pad 6: unconnected-(J2-Pin_6-Pad6) -> Net-(U2-USB_DP_DN1)
- U2 pad A13: unconnected-(U2-USB_DM_DN2-PadA13) -> Net-(U2-USB_DM_DN2)
- U2 pad A20: unconnected-(U2-USB_DP_DN1-PadA20) -> Net-(U2-USB_DP_DN1)
- U2 pad B12: unconnected-(U2-USB_DP_DN2-PadB12) -> Net-(U2-USB_DP_DN2)
- U2 pad B18: unconnected-(U2-USB_DM_DN1-PadB18) -> Net-(U2-USB_DM_DN1)
Routing:
- net Net-(U2-USB_DM_DN1): track 0.00 -> 42.1 mm, vias 0 -> 1
- net Net-(U2-USB_DP_DN1): track 0.00 -> 42.1 mm, vias 0 -> 1
- net GND: track 38.3 -> 2.59 mm
- net Net-(U2-USB_DM_DN2): track 0.00 -> 30.0 mm, vias 0 -> 1
- net Net-(U2-USB_DP_DN2): track 0.00 -> 30.0 mm, vias 0 -> 1
- net +5V: track 12.7 -> 13.9 mm
- added copper zone on F.Cu, net GND

Commit message: Updated PCB Design
Signed-off-by: Jakub Sobota <jakub.sobota@3mdeb.com>
Parts:
- removed U$1: M.2-B+M-KEY, M.2:M.2-B+M-KEY
- added C10: 0.1 μF, Capacitor_SMD:C_0402_1005Metric_Pad0.74x0.62mm_HandSolder, F.Cu at (128.5, 104.5)
- added C11: 0.1 μF, Capacitor_SMD:C_0402_1005Metric_Pad0.74x0.62mm_HandSolder, F.Cu at (128.6, 109.3)
- added C12: 150uF, Capacitor_SMD:CP_Elec_6.3x5.9, F.Cu at (152.8, 95.5)
- added C13: 150uF, Capacitor_SMD:CP_Elec_6.3x5.9, F.Cu at (139.4, 95.5)
- added C14: 0.1uF, Capacitor_SMD:C_0402_1005Metric_Pad0.74x0.62mm_HandSolder, F.Cu at (143.0, 123.9)
- added C15: 0.1uF, Capacitor_SMD:C_0402_1005Metric_Pad0.74x0.62mm_HandSolder, F.Cu at (143.0, 122.9)
- added C16: 1000pF, Capacitor_SMD:C_0402_1005Metric_Pad0.74x0.62mm_HandSolder, F.Cu at (140.0, 123.6)
- added C17: 22 µF, Capacitor_SMD:C_0402_1005Metric_Pad0.74x0.62mm_HandSolder, B.Cu at (141.0, 123.1)
- added C18: 22 µF, Capacitor_SMD:C_0402_1005Metric_Pad0.74x0.62mm_HandSolder, B.Cu at (140.0, 123.1)
- added C19: 22 µF, Capacitor_SMD:C_0402_1005Metric_Pad0.74x0.62mm_HandSolder, B.Cu at (139.0, 123.1)
- added C20: 22 µF, Capacitor_SMD:C_0402_1005Metric_Pad0.74x0.62mm_HandSolder, B.Cu at (138.0, 123.1)
- added C21: 22 µF, Capacitor_SMD:C_0402_1005Metric_Pad0.74x0.62mm_HandSolder, B.Cu at (137.0, 123.1)
- added C22: 0.01 μF, Capacitor_SMD:C_0402_1005Metric_Pad0.74x0.62mm_HandSolder, B.Cu at (145.9, 120.0)
- added C23: 0.1 μF, Capacitor_SMD:C_0402_1005Metric_Pad0.74x0.62mm_HandSolder, B.Cu at (145.9, 119.0)
- added C24: 0.1 μF, Capacitor_SMD:C_0402_1005Metric_Pad0.74x0.62mm_HandSolder, B.Cu at (145.9, 118.1)
- added C25: 0.01 μF, Capacitor_SMD:C_0402_1005Metric_Pad0.74x0.62mm_HandSolder, B.Cu at (145.9, 117.2)
- added C26: 0.1 μF, Capacitor_SMD:C_0402_1005Metric_Pad0.74x0.62mm_HandSolder, B.Cu at (145.9, 116.2)
- added C27: 0.1 μF, Capacitor_SMD:C_0402_1005Metric_Pad0.74x0.62mm_HandSolder, B.Cu at (148.1, 120.0)
- added C28: 0.01 μF, Capacitor_SMD:C_0402_1005Metric_Pad0.74x0.62mm_HandSolder, B.Cu at (148.1, 119.1)
- added C29: 0.1 μF, Capacitor_SMD:C_0402_1005Metric_Pad0.74x0.62mm_HandSolder, B.Cu at (148.1, 118.1)
- added C30: 0.1 μF, Capacitor_SMD:C_0402_1005Metric_Pad0.74x0.62mm_HandSolder, B.Cu at (148.1, 117.2)
- added C31: 0.01 μF, Capacitor_SMD:C_0402_1005Metric_Pad0.74x0.62mm_HandSolder, B.Cu at (148.1, 116.2)
- added C32: 0.1 μF, Capacitor_SMD:C_0402_1005Metric_Pad0.74x0.62mm_HandSolder, B.Cu at (150.3, 120.0)
- added C33: 0.1 μF, Capacitor_SMD:C_0402_1005Metric_Pad0.74x0.62mm_HandSolder, B.Cu at (150.3, 119.1)
- added C34: 22 μF, Capacitor_SMD:C_0805_2012Metric_Pad1.18x1.45mm_HandSolder, B.Cu at (147.3, 123.0)
- added C35: 18pF, Capacitor_SMD:C_0402_1005Metric_Pad0.74x0.62mm_HandSolder, F.Cu at (147.8, 112.7)
- added C36: 18pF, Capacitor_SMD:C_0402_1005Metric_Pad0.74x0.62mm_HandSolder, F.Cu at (148.7, 111.7)
- added C37: 0.01 μF, Capacitor_SMD:C_0402_1005Metric_Pad0.74x0.62mm_HandSolder, B.Cu at (150.3, 118.1)
- added C38: 0.1 μF, Capacitor_SMD:C_0402_1005Metric_Pad0.74x0.62mm_HandSolder, B.Cu at (150.3, 117.2)
- added C39: 0.1 μF, Capacitor_SMD:C_0402_1005Metric_Pad0.74x0.62mm_HandSolder, B.Cu at (150.3, 116.2)
- added C40: 0.01 μF, Capacitor_SMD:C_0402_1005Metric_Pad0.74x0.62mm_HandSolder, B.Cu at (152.5, 116.2)
- added C41: 0.1 μF, Capacitor_SMD:C_0402_1005Metric_Pad0.74x0.62mm_HandSolder, B.Cu at (152.5, 117.2)
- added C42: 0.1 μF, Capacitor_SMD:C_0402_1005Metric_Pad0.74x0.62mm_HandSolder, B.Cu at (152.5, 118.1)
- added C43: 0.01 μF, Capacitor_SMD:C_0402_1005Metric_Pad0.74x0.62mm_HandSolder, B.Cu at (152.5, 119.1)
- added C44: 0.1 μF, Capacitor_SMD:C_0402_1005Metric_Pad0.74x0.62mm_HandSolder, B.Cu at (152.5, 120.0)
- added C45: 0.1 μF, Capacitor_SMD:C_0402_1005Metric_Pad0.74x0.62mm_HandSolder, F.Cu at (161.2, 118.1)
- added C46: 0.01 μF, Capacitor_SMD:C_0402_1005Metric_Pad0.74x0.62mm_HandSolder, F.Cu at (162.1, 106.5)
- added C47: 0.1 μF, Capacitor_SMD:C_0402_1005Metric_Pad0.74x0.62mm_HandSolder, F.Cu at (162.1, 108.5)
- added C48: 0.1 μF, Capacitor_SMD:C_0402_1005Metric_Pad0.74x0.62mm_HandSolder, F.Cu at (162.1, 110.4)
- added C49: 0.01 μF, Capacitor_SMD:C_0402_1005Metric_Pad0.74x0.62mm_HandSolder, F.Cu at (162.1, 112.4)
- added C50: 0.1 μF, Capacitor_SMD:C_0402_1005Metric_Pad0.74x0.62mm_HandSolder, F.Cu at (165.4, 100.6)
- added C51: 0.1 μF, Capacitor_SMD:C_0402_1005Metric_Pad0.74x0.62mm_HandSolder, F.Cu at (165.4, 102.6)
- added C52: 0.1 μF, Capacitor_SMD:C_0402_1005Metric_Pad0.74x0.62mm_HandSolder, F.Cu at (165.4, 104.5)
- added C53: 0.1 μF, Capacitor_SMD:C_0402_1005Metric_Pad0.74x0.62mm_HandSolder, F.Cu at (165.4, 106.5)
- added C54: 0.1 μF, Capacitor_SMD:C_0402_1005Metric_Pad0.74x0.62mm_HandSolder, F.Cu at (165.4, 108.5)
- added C55: 0.1 μF, Capacitor_SMD:C_0402_1005Metric_Pad0.74x0.62mm_HandSolder, F.Cu at (165.4, 110.4)
- added C56: 22 μF, Capacitor_SMD:C_0805_2012Metric_Pad1.18x1.45mm_HandSolder, F.Cu at (170.5, 115.8)
- added C57: 0.01 μF, Capacitor_SMD:C_0402_1005Metric_Pad0.74x0.62mm_HandSolder, F.Cu at (165.4, 112.4)
- added C9: 0.1 μF, Capacitor_SMD:C_0402_1005Metric_Pad0.74x0.62mm_HandSolder, F.Cu at (131.9, 103.7)
- added D6: LED, LED_SMD:LED_0603_1608Metric_Pad1.05x0.95mm_HandSolder, F.Cu at (124.7, 97.4)
- added D7: LED, LED_SMD:LED_0603_1608Metric_Pad1.05x0.95mm_HandSolder, F.Cu at (124.6, 94.4)
- added FB1: 220 Ohm, Inductor_SMD:L_0603_1608Metric_Pad1.05x0.95mm_HandSolder, F.Cu at (169.8, 111.8)
- added FL1: 90 Ohm, Filters:MCZ1210AH_CP, B.Cu at (140.9, 100.0)
- added FL2: 90 Ohm, Filters:MCZ1210AH_CP, B.Cu at (150.2, 100.1)
- added J1: ~, M2_Edge_connector:M.2_KEY_M_B, F.Cu at (146.2, 130.6)
- added R10: 9.09 KOhm, Resistor_SMD:R_0402_1005Metric_Pad0.72x0.64mm_HandSolder, F.Cu at (145.3, 112.9)
- added R11: NOPOP, Resistor_SMD:R_0402_1005Metric_Pad0.72x0.64mm_HandSolder, F.Cu at (153.1, 125.0)
- added R12: NOPOP, Resistor_SMD:R_0402_1005Metric_Pad0.72x0.64mm_HandSolder, F.Cu at (152.1, 125.0)
- added R13: NOPOP, Resistor_SMD:R_0402_1005Metric_Pad0.72x0.64mm_HandSolder, F.Cu at (150.2, 125.0)
- added R14: NOPOP, Resistor_SMD:R_0402_1005Metric_Pad0.72x0.64mm_HandSolder, F.Cu at (151.2, 125.0)
- added R15: NOPOP, Resistor_SMD:R_0402_1005Metric_Pad0.72x0.64mm_HandSolder, F.Cu at (120.4, 97.9)
- added R16: NOPOP, Resistor_SMD:R_0402_1005Metric_Pad0.72x0.64mm_HandSolder, F.Cu at (129.2, 101.8)
- added R17: 30.9 KOhm, Resistor_SMD:R_0402_1005Metric_Pad0.72x0.64mm_HandSolder, F.Cu at (120.3, 104.8)
- added R18: 10 KOhm, Resistor_SMD:R_0402_1005Metric_Pad0.72x0.64mm_HandSolder, F.Cu at (123.5, 100.9)
- added R19: 10 KOhm, Resistor_SMD:R_0402_1005Metric_Pad0.72x0.64mm_HandSolder, F.Cu at (120.3, 101.9)
- added R20: 680 Ohm, Resistor_SMD:R_0402_1005Metric_Pad0.72x0.64mm_HandSolder, F.Cu at (125.9, 102.3)
- added R21: 680 Ohm, Resistor_SMD:R_0402_1005Metric_Pad0.72x0.64mm_HandSolder, F.Cu at (123.9, 105.4)
- added R22: NOPOP, Resistor_SMD:R_0402_1005Metric_Pad0.72x0.64mm_HandSolder, F.Cu at (155.4, 122.9)
- added R23: 10 KOhm, Resistor_SMD:R_0402_1005Metric_Pad0.72x0.64mm_HandSolder, F.Cu at (155.4, 123.8)
- added R24: 0 Ohm, LED_SMD:LED_0402_1005Metric_Pad0.77x0.64mm_HandSolder, F.Cu at (155.4, 122.0)
- added R25: 0 Ohm, LED_SMD:LED_0402_1005Metric_Pad0.77x0.64mm_HandSolder, F.Cu at (155.4, 121.0)
- added R26: 4.7 KOhm, Resistor_SMD:R_0402_1005Metric_Pad0.72x0.64mm_HandSolder, F.Cu at (153.6, 112.2)
- added R27: 1 MOhm, Resistor_SMD:R_0402_1005Metric_Pad0.72x0.64mm_HandSolder, F.Cu at (146.5, 111.7)
- added R28: 0 Ohm, Resistor_SMD:R_0402_1005Metric_Pad0.72x0.64mm_HandSolder, F.Cu at (140.0, 124.6)
- added U4: TPS2560, Package_SON:VSON-10-1EP_3x3mm_P0.5mm_EP1.65x2.4mm_ThermalVias, F.Cu at (139.5, 103.5)
- added Y2: 48 MHz, Crystal:Crystal_SMD_Abracon_ABM3B-4Pin_5.0x3.2mm, F.Cu at (147.5, 109.0)
- C1, C2, C3, D1, D2, D4, F1, F2, R1, R2, R3, R4: moved to B.Cu
- C6: moved to F.Cu
- D3: footprint Diode_SMD:D_SOD-523 -> Diode_SMD:D_SOD-323_HandSoldering; moved to B.Cu
- U1: footprint DC-DC_Converter:TPS61023 -> DC-DC:TPS61023; moved to B.Cu
- U2: footprint TUSB7320:Texas_tusb7340 -> TUSB7320:Texas_tusb7320
- moved R1 36.4 mm to (173.2, 107.6)
- moved R2 34.4 mm to (171.6, 112.2), turned to 180 degrees
- moved D2 33.6 mm to (172.7, 110.0), turned to 180 degrees
- moved C2 31.3 mm to (170.3, 103.2)
- moved R3 29.4 mm to (165.0, 109.6), turned to 180 degrees
- moved D1 27.1 mm to (160.4, 106.6), turned to 180 degrees
- moved F2 26.2 mm to (164.8, 106.7), turned to 180 degrees
- moved C3 25.5 mm to (164.7, 102.6)
- moved R4 24.6 mm to (165.0, 111.6), turned to 180 degrees
- moved C1 24.5 mm to (160.4, 102.7), turned to 180 degrees
- moved D4 21.9 mm to (160.0, 109.6)
- moved F3 17.2 mm to (137.5, 114.9), turned to 90 degrees
- moved R8 15.7 mm to (137.6, 107.1), turned to 0 degrees
- moved U1 14.9 mm to (154.2, 107.9), turned to 180 degrees
- moved C8 14.9 mm to (139.9, 106.8), turned to 180 degrees
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Connections:
- C1 pad 1: Net-(D1-A) -> +3.3V
- D1 pad 2: Net-(D1-A) -> +3.3V
- D3 pad 1: Net-(D1-A) -> GND
- D3 pad 2: GND -> +3.3V
- F1 pad 1: +3.3V -> Net-(C17-Pad1)
- F1 pad 2: Net-(D1-A) -> +3.3V
- J2 pad 1: +5V -> DS1_VBUS
- J2 pad 2: +5V -> DS2_VBUS
- J2 pad 3: Net-(U2-USB_DM_DN2) -> Net-(FL2-Pad4)
- J2 pad 4: Net-(U2-USB_DM_DN1) -> Net-(FL1-Pad1)
- J2 pad 5: Net-(U2-USB_DP_DN2) -> Net-(FL2-Pad3)
- J2 pad 6: Net-(U2-USB_DP_DN1) -> Net-(FL1-Pad2)
- L1 pad 1: Net-(D1-A) -> +3.3V
- U1 pad 2: Net-(D1-A) -> +3.3V
- U1 pad 3: Net-(D1-A) -> +3.3V
- U2 pad A1: unconnected-(U2-VDD11-PadA1) -> +1.1V
- U2 pad A12: unconnected-(U2-VDD11-PadA12) -> +1.1V
- U2 pad A13: Net-(U2-USB_DM_DN2) -> DM2
- U2 pad A15: unconnected-(U2-GRST#-PadA15) -> GRSTZ
- U2 pad A16: unconnected-(U2-VDD11-PadA16) -> +1.1V
- U2 pad A19: unconnected-(U2-VDDA_3P3-PadA19) -> VDDA_3P3
- U2 pad A2: unconnected-(U2-SDA-PadA2) -> Net-(U2-SDA)
- U2 pad A20: Net-(U2-USB_DP_DN1) -> DP1
- U2 pad A21: unconnected-(U2-VDDA_3P3-PadA21) -> VDDA_3P3
- U2 pad A22: unconnected-(U2-XO-PadA22) -> Net-(U2-XO)
- U2 pad A23: unconnected-(U2-XI-PadA23) -> Net-(U2-XI)
- U2 pad A24: unconnected-(U2-R1EXT-PadA24) -> Net-(U2-R1EXT)
- U2 pad A25: unconnected-(U2-VDDA_3P3-PadA25) -> VDDA_3P3
- U2 pad A28: unconnected-(U2-VDD11-PadA28) -> +1.1V
- U2 pad A3: unconnected-(U2-VDD33-PadA3) -> +3.3V
- U2 pad A31: unconnected-(U2-VDD11-PadA31) -> +1.1V
- U2 pad A33: unconnected-(U2-VDD11-PadA33) -> +1.1V
- U2 pad A34: unconnected-(U2-VDD33-PadA34) -> +3.3V
- U2 pad A36: unconnected-(U2-OVERCUR1#-PadA36) -> OVERCUR1Z
- U2 pad A37: unconnected-(U2-OVERCUR2#-PadA37) -> OVERCUR2Z
- U2 pad A38: unconnected-(U2-VDD11-PadA38) -> +1.1V
- U2 pad A39: unconnected-(U2-VDD33-PadA39) -> +3.3V
- U2 pad A4: unconnected-(U2-VDD11-PadA4) -> +1.1V
- U2 pad A40: unconnected-(U2-PERST#-PadA40) -> PERSTZ
- U2 pad A41: unconnected-(U2-PCIE_TXN-PadA41) -> PCIE_TXN
- U2 pad A42: unconnected-(U2-PCIE_RXN-PadA42) -> PCIE_RXN
- U2 pad A44: unconnected-(U2-VDDA_3P3-PadA44) -> VDDA_3P3
- U2 pad A45: unconnected-(U2-PCIE_REFCLKP-PadA45) -> PCIE_REFCLKP
- U2 pad A47: unconnected-(U2-VDD33-PadA47) -> +3.3V
- U2 pad A49: unconnected-(U2-GPIO0-PadA49) -> Net-(U2-GPIO0)
- U2 pad A50: unconnected-(U2-VDD11-PadA50) -> +1.1V
- U2 pad A51: unconnected-(U2-VDD33-PadA51) -> +3.3V
- U2 pad A52: unconnected-(U2-AUX_DET-PadA52) -> Net-(U2-AUX_DET)
- U2 pad A6: unconnected-(U2-VDD11-PadA6) -> +1.1V
- U2 pad A9: unconnected-(U2-VDD11-PadA9) -> +1.1V
- U2 pad B1: unconnected-(U2-VDD11-PadB1) -> +1.1V
- U2 pad B11: unconnected-(U2-VDDA_3P3-PadB11) -> VDDA_3P3
- U2 pad B12: Net-(U2-USB_DP_DN2) -> DP2
- U2 pad B14: unconnected-(U2-FREQSEL-PadB14) -> Net-(U2-FREQSEL)
- U2 pad B17: unconnected-(U2-VDD11-PadB17) -> +1.1V
- U2 pad B18: Net-(U2-USB_DM_DN1) -> DM1
- U2 pad B19: unconnected-(U2-VDD11-PadB19) -> +1.1V
- U2 pad B2: unconnected-(U2-SCL-PadB2) -> Net-(U2-SCL)
- U2 pad B21: unconnected-(U2-VSS_OSC-PadB21) -> Net-(U2-VSS_OSC)
- U2 pad B22: unconnected-(U2-VDDA_3P3-PadB22) -> VDDA_3P3
- U2 pad B23: unconnected-(U2-R1EXTRTN-PadB23) -> Net-(U2-R1EXTRTN)
- U2 pad B24: unconnected-(U2-VDD11-PadB24) -> +1.1V
- U2 pad B32: unconnected-(U2-JTAG_RST#-PadB32) -> GND
- U2 pad B33: unconnected-(U2-PWRON1#-PadB33) -> PWRON1Z
- U2 pad B34: unconnected-(U2-PWRON2#-PadB34) -> PWRON2Z
- U2 pad B35: unconnected-(U2-WAKE#-PadB35) -> WAKEZ
- U2 pad B37: unconnected-(U2-VDD11-PadB37) -> +1.1V
- U2 pad B38: unconnected-(U2-PCIE_TXP-PadB38) -> PCIE_TXP
- U2 pad B39: unconnected-(U2-PCIE_RXP-PadB39) -> PCIE_RXP
- U2 pad B40: unconnected-(U2-VDD11-PadB40) -> +1.1V
- U2 pad B41: unconnected-(U2-PCIE_REFCLKN-PadB41) -> PCIE_REFCLKN
- U2 pad B42: unconnected-(U2-VDD11-PadB42) -> +1.1V
- U2 pad B44: unconnected-(U2-VDD11-PadB44) -> +1.1V
- U2 pad B46: unconnected-(U2-GPIO1-PadB46) -> Net-(U2-GPIO1)
- U2 pad B47: unconnected-(U2-GPIO2-PadB47) -> Net-(U2-GPIO2)
- U2 pad B48: unconnected-(U2-GPIO3-PadB48) -> Net-(U2-GPIO3)
Routing:
- net +1.1V: track 0.00 -> 61.9 mm, vias 1 -> 16
- net Net-(U2-USB_DM_DN1): track 42.1 -> 0.00 mm, vias 1 -> 0
- net Net-(U2-USB_DP_DN1): track 42.1 -> 0.00 mm, vias 1 -> 0
- net Net-(C17-Pad1): track 0.00 -> 40.6 mm, vias 0 -> 1
- net Net-(U2-USB_DM_DN2): track 30.0 -> 0.00 mm, vias 1 -> 0
- net Net-(U2-USB_DP_DN2): track 30.0 -> 0.00 mm, vias 1 -> 0
- net Net-(D5-A): track 0.53 -> 26.4 mm, vias 1 -> 3
- net +5V: track 13.9 -> 0.00 mm, vias 4 -> 0
- net +3.3V: track 0.52 -> 12.7 mm, vias 5 -> 0
- net PCIE_REFCLKP: track 0.00 -> 10.7 mm
- net Net-(U2-XO): track 0.00 -> 10.5 mm
- net GND: track 2.59 -> 11.8 mm, vias 53 -> 35
- net Net-(U1-SW): track 8.79 -> 0.00 mm
- net WAKEZ: track 0.00 -> 8.58 mm, vias 0 -> 2
- net GRSTZ: track 9.15 -> 3.21 mm, vias 2 -> 1
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- removed copper zone on B.Cu, net +3.3V
- removed copper zone on In1.Cu, net GND
- removed copper zone on In2.Cu, net GND
- removed copper zone on B.Cu, net Net-(D5-A)
Other:
- outline, holes or cut-outs redrawn
