File: Kicad-Files/PCI2USB.kicad_pcb (KiCad board)
At the start: 4 copper layers, 22 x 80 mm, 104 parts, among them IC1 TUSB7320, J1 M.2 Edge Connector, J2 USB_9PIN_Internal, U1 TPS61023DRLR, U2 TPS2560DRC, U3 TPS74401, Y1 48 MHz

Commit message: Updated 3D models and Logo
Signed-off-by: Jakub Sobota <jakub.sobota@3mdeb.com>
Parts:
- added G***: LOGO, LOGO, F.Cu at (140.8, 124.5)
- moved C50 4.70 mm to (155.1, 118.4)
- moved C46 0.94 mm to (155.1, 122.2)
- moved C48 0.94 mm to (155.1, 120.3)
- moved C49 0.94 mm to (155.1, 119.3)
- moved C45 0.94 mm to (155.1, 123.1)
- moved C47 0.94 mm to (155.1, 121.2)
- moved R28 0.15 mm to (150.2, 116.8)
- moved C16 0.15 mm to (150.2, 117.8)
Connections:
- net D1+ renamed DP1
- net D1- renamed DM1
- net D2+ renamed DP2
- net D2- renamed DM2
- net Net-(J1-PERn0/SATA-B+) renamed SATA-B+
- net Net-(J1-PERp0/SATA-B-) renamed SATA-B-
Routing:
- net Net-(U3-BIAS): track 16.4 -> 19.0 mm

Commit message: Moved USB connector to acheive wider 5V traces
Signed-off-by: Jakub Sobota <jakub.sobota@3mdeb.com>
Parts:
- moved J2 0.38 mm to (150.3, 95.0)
Connections:
- net SATA-B+ renamed Net-(J1-PERn0/SATA-B+)
- net SATA-B- renamed Net-(J1-PERp0/SATA-B-)
Routing:
- net DS2_VBUS: track 22.7 -> 21.4 mm

Commit message: fixed pdf schematics, removed temporary files
Signed-off-by: Jakub Sobota <jakub.sobota@3mdeb.com>
Connections:
- D8 pad 4: DP1 -> DM1
- D8 pad 5: DM1 -> DP1
Changed lines of the file:
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@@
 		(tags "capacitor handsolder")
 		(property "Reference" "C11"
-			(at -1.43 -0.51 0)
+			(at -1.43 -0.5227 0)
 			(layer "F.SilkS")
 			(effects
@@
 			(layers "F.Cu" "F.Mask" "F.Paste")
 			(net 133 "DP2")
-			(pinfunction "I/O2")
+			(pinfunction "I/O3")
 			(pintype "passive")
 		)
 		(pad "4" smd rect
-			(at 1.25 0.95 270)
+			(at 1.25 -0.95 270)
 			(size 0.6 1.2)
 			(layers "F.Cu" "F.Mask" "F.Paste")
-			(net 135 "DP1")
-			(pinfunction "I/O3")
+			(net 134 "DM1")
+			(pinfunction "I/O4")
 			(pintype "passive")
 		)
 		(pad "5" smd rect
-			(at 1.25 -0.95 270)
+			(at 1.25 0.95 270)
 			(size 0.6 1.2)
 			(layers "F.Cu" "F.Mask" "F.Paste")
-			(net 134 "DM1")
-			(pinfunction "I/O4")
+			(net 135 "DP1")
+			(pinfunction "I/O5")
 			(pintype "passive")
 		)
@@
 		(tags "resistor handsolder")
 		(property "Reference" "R21"
-			(at -1.46 0.0408 180)
+			(at -1.46 0.0281 180)
 			(layer "F.SilkS")
 			(effects
@@
 		(tags "capacitor handsolder")
 		(property "Reference" "C20"
-			(at -1.778 0 90)
+			(at -1.778 -0.1016 90)
 			(layer "B.SilkS")
 			(effects

Commit message: Created all necessary production files
Signed-off-by: Jakub Sobota <jakub.sobota@3mdeb.com>
Routing:
- net VDDA_3P3: track 52.7 -> 57.3 mm
- net +1.1V: track 134.2 -> 136.2 mm
- added copper zone on In2.Cu, net GND

Commit message: Added more thermal relief points, and bigger power traces
Signed-off-by: Jakub Sobota <jakub.sobota@3mdeb.com>
Routing:
- net Net-(C17-Pad1): track 68.2 -> 62.3 mm
- net GND: vias 100 -> 111

Commit message: Updated all SMD footprints to not hand soldered versions
Signed-off-by: Jakub Sobota <jakub.sobota@3mdeb.com>
Parts:
- C1, C2, C3, C34, C4, C56, C7: footprint Capacitor_SMD:C_0805_2012Metric_Pad1.18x1.45mm_HandSolder -> Capacitor_SMD:C_0805_2012Metric
- C10, C11, C17, C18, C19, C20, C21, C22, C23, C24, C25, C26, C27, C28, C29, C30, C31, C32, C33, C35, C36, C37, C38, C39, C40, C41, C42, C43, C44, C45, C46, C47, C48, C49, C50, C51, C52, C53, C54, C55, C57, C6, C8, C9: footprint Capacitor_SMD:C_0402_1005Metric_Pad0.74x0.62mm_HandSolder -> Capacitor_SMD:C_0402_1005Metric
- D4, D6, D7: footprint LED_SMD:LED_0603_1608Metric_Pad1.05x0.95mm_HandSolder -> LED_SMD:LED_0603_1608Metric
- F1, F2, F3: footprint Fuse:Fuse_0603_1608Metric_Pad1.05x0.95mm_HandSolder -> Fuse:Fuse_0603_1608Metric
- FB1: footprint Inductor_SMD:L_0603_1608Metric_Pad1.05x0.95mm_HandSolder -> Inductor_SMD:L_0603_1608Metric
- R1: footprint Resistor_SMD:R_0603_1608Metric_Pad0.98x0.95mm_HandSolder -> Resistor_SMD:R_0603_1608Metric
- R10, R17, R18, R19, R2, R20, R21, R23, R24, R25, R26, R27, R28, R29, R4, R5, R6, R7, R8: footprint Resistor_SMD:R_0402_1005Metric_Pad0.72x0.64mm_HandSolder -> Resistor_SMD:R_0402_1005Metric
