File: Kicad-Files/PCI2USB.kicad_sch (KiCad schematic)
At the start: 15 parts, among them U1 TPS61023

Commit message: Updated schematics and board layout
Signed-off-by: Jakub Sobota <jakub.sobota@3mdeb.com>
Parts:
- removed D3: 4V/5A, Diode_SMD:D_SOD-523, symbol Diode:PTVS5V0Z1USK
- removed D4: LED, LED_SMD:LED_0603_1608Metric_Pad1.05x0.95mm_HandSolder, symbol Device:LED
- added D3: LED, LED_SMD:LED_0603_1608Metric_Pad1.05x0.95mm_HandSolder, symbol Device:LED
- added D4: 6V/5A, Diode_SMD:D_SOD-523, symbol Diode:PTVS5V0Z1USK
- added J1: Bus_M.2_Socket_B, symbol Connector:Bus_M.2_Socket_B
- added J2: USB 9 Pin Connecetor, Connectors:USB 9 Pin internal header, symbol Connector:Conn_01x09_Pin
- D2: value 6V/5A -> 4V/5A
- R1: value 732 KOhm -> 680 Ohm; footprint Resistor_SMD:R_0603_1608Metric_Pad0.98x0.95mm_HandSolder -> Resistor_SMD:R_0201_0603Metric_Pad0.64x0.40mm_HandSolder
- R3: value 680 Ohm -> 732 KOhm; footprint Resistor_SMD:R_0201_0603Metric_Pad0.64x0.40mm_HandSolder -> Resistor_SMD:R_0603_1608Metric_Pad0.98x0.95mm_HandSolder
Connections:
- net +5V: now also J2.1 (Pin_1), J2.2 (Pin_2)
- net GND: now also R1.2, D4.2 (A), J2.7 (Pin_7), J2.8 (Pin_8); no longer R3.2
- net at C2.2, C3.2, F2.1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: now also R3.2, D3.2 (A), D4.1 (K); no longer D2.1 (K), R1.2
- net at C1.1, D1.2 (A), F1.2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: now also D2.1 (K)
- net at R4.1: now also D3.1 (K)
- net at R2.2, U1.1 (FB): now also R3.1; no longer R1.1
- net at D1.1 (K): now also R1.1; no longer R3.1
- new net: J1.11 (GND), J1.27 (GND), J1.3 (GND), J1.33 (GND), J1.39 (GND), J1.45 (GND), J1.5 (GND), J1.51 (GND), J1.57 (GND), J1.71 (GND), J1.73 (GND)
- new net VIN: J1.2 (3.3V), J1.4 (3.3V), J1.70 (3.3V), J1.72 (3.3V), J1.74 (3.3V)
Other:
- added sheet Power Section (Power Section.kicad_sch)
- added sheet Signals (Signals.kicad_sch)
- title: m2 PCIe to USB Converter -> PCI2USB

Commit message: Created schematics for 1.1V circuit
Signed-off-by: Jakub Sobota <jakub.sobota@3mdeb.com>
Parts:
- removed C1: 10 μF, Capacitor_SMD:C_0805_2012Metric_Pad1.18x1.45mm_HandSolder, symbol Device:C_Small
- removed C2, C3: 22 μF, Capacitor_SMD:C_1206_3216Metric_Pad1.33x1.80mm_HandSolder, symbol Device:C_Small
- removed D1, D3: LED, LED_SMD:LED_0603_1608Metric_Pad1.05x0.95mm_HandSolder, symbol Device:LED
- removed D2: 4V/5A, Diode_SMD:D_SOD-523, symbol Diode:PTVS5V0Z1USK
- removed D4: 6V/5A, Diode_SMD:D_SOD-523, symbol Diode:PTVS5V0Z1USK
- removed F1: 4A, Fuse:Fuse_0603_1608Metric_Pad1.05x0.95mm_HandSolder, symbol Device:Fuse_Small
- removed F2: 5A, Fuse:Fuse_0603_1608Metric_Pad1.05x0.95mm_HandSolder, symbol Device:Fuse_Small
- removed L1: 1 μH, Inductor_SMD:L_Chilisin_BMRx00050515, symbol Device:L
- removed R1: 680 Ohm, Resistor_SMD:R_0201_0603Metric_Pad0.64x0.40mm_HandSolder, symbol Device:R_US
- removed R2: 100 KOhm, Resistor_SMD:R_0603_1608Metric_Pad0.98x0.95mm_HandSolder, symbol Device:R_US
- removed R3: 732 KOhm, Resistor_SMD:R_0603_1608Metric_Pad0.98x0.95mm_HandSolder, symbol Device:R_US
- removed R4: 1.5 KOhm, Resistor_SMD:R_0201_0603Metric_Pad0.64x0.40mm_HandSolder, symbol Device:R_US
- removed U1: TPS61023, DC-DC_Converter:TPS61023, symbol TPS61023:TPS61023
Other:
- sheet Power Section renamed USB Power
- sheet Signals renamed TUSB7320 (page 2)
- added sheet 1.1V Regulator (untitled.kicad_sch)

Commit message: Created 1.1V Circuit for USB Host IC
Signed-off-by: Jakub Sobota <jakub.sobota@3mdeb.com>
Other:
- sheet TUSB7320 (page 2) renamed TUSB7320
Changed lines of the file:
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@@
 			(color 0 0 0 0.0000)
 		)
-		(property "Sheetname" "TUSB7320 (page 2)"
+		(property "Sheetname" "TUSB7320"
 			(at 40.64 -14.6816 0)
 			(effects

Commit message: Fixed signal integrity for USB data lines
Signed-off-by: Jakub Sobota <jakub.sobota@3mdeb.com>
Parts:
- removed J2: USB 9 Pin Connecetor, Connectors:USB 9 Pin internal header, symbol Connector:Conn_01x09_Pin

Commit message: Created schematics for TUSB7320 USB Controller
Signed-off-by: Jakub Sobota <jakub.sobota@3mdeb.com>
Parts:
- removed J1: Bus_M.2_Socket_B, symbol Connector:Bus_M.2_Socket_B
- added J2: USB_9PIN_Internal, Connectors:USB 9 Pin internal header, symbol Connectors:USB_9PIN_Internal
- added J3: ~, M2_Edge_connector:M.2_KEY_M_B, symbol M2_Edge_connector:M.2_Key_M_B
Connections:
- new net DM1: J2.3 (D-)
- new net DM2: J2.6 (D+)
- new net DP1: J2.5 (D+)
- new net DP2: J2.4 (D-)
- new net DS1_VBUS: J2.1 (5V)
- new net DS2_VBUS: J2.2 (5V)
- new net GND: J2.7 (GND), J2.8 (GND)
Other:
- sheet 1.1V Regulator renamed TUSB7320 Power
- sheet TUSB7320: file Signals.kicad_sch -> USBController.kicad_sch
- sheet TUSB7320 Power: file untitled.kicad_sch -> TUSB7320 Power.kicad_sch
- sheet USB Power: file Power Section.kicad_sch -> USB Power.kicad_sch

Commit message: Complete Schematics and BOM
Signed-off-by: Jakub Sobota <jakub.sobota@3mdeb.com>
Parts:
- added C14, C15: 0.1uF, Capacitor_SMD:C_0402_1005Metric_Pad0.74x0.62mm_HandSolder, symbol Device:C_Small
- added C16: 1000pF, Capacitor_SMD:C_0402_1005Metric_Pad0.74x0.62mm_HandSolder, symbol Device:C_Small
- added C17, C18, C19, C20, C21: 22 µF, Capacitor_SMD:C_0402_1005Metric_Pad0.74x0.62mm_HandSolder, symbol Device:C_Small
- added D3: 4V/5A, Diode_SMD:D_SOD-323_HandSoldering, symbol Diode:PTVS5V0Z1USK
- added F1: 5A, Fuse:Fuse_0603_1608Metric_Pad1.05x0.95mm_HandSolder, symbol Device:Fuse_Small
- added FL1, FL2: 90 Ohm, Filters:MCZ1210AH_CP, symbol Filter:Choke_CommonMode_PulseElectronics_PH9455x405NL
- added R28: 0 Ohm, Resistor_SMD:R_0402_1005Metric_Pad0.72x0.64mm_HandSolder, symbol Device:R_Small_US
- renumbered J3 to J1
Connections:
- net DM1: now also FL2.1; no longer J2.3 (D-)
- net DM2: now also FL1.2; no longer J2.6 (D+)
- net DP1: now also FL2.2; no longer J2.5 (D+)
- net DP2: now also FL1.1; no longer J2.4 (D-)
- net GND: now also J1.27 (GND), J1.3 (GND), J1.33 (GND), J1.39 (GND), J1.45 (GND), J1.51 (GND), J1.57 (GND), J1.71 (GND), J1.73 (GND), C16.1, C17.2, C18.2, C19.2, C20.2, C21.2, D3.1 (K)
- net PCIE_REFCLKN: now also J1.53 (REFCLKn)
- net PCIE_REFCLKP: now also J1.55 (REFCLKp)
- net PCIE_RXN: now also J1.49 (PETp0/SATA-A+)
- net PCIE_RXP: now also J1.47 (PETn0/SATA-A-)
- net PCIE_TXN: now also C15.2
- net PCIE_TXP: now also C14.2
- net PERSTZ: now also J1.50 (PERST#)
- net WAKEZ: now also C16.2, R28.1
- net at J1.2 (3.3V): now also J1.4 (3.3V), J1.70 (3.3V), J1.72 (3.3V), J1.74 (3.3V), C17.1, C18.1, C19.1, C20.1, C21.1, F1.1
- net at J1.41 (PERn0/SATA-B+): now also C14.1
- net at J1.43 (PERp0/SATA-B-): now also C15.1
- net at J1.54 (PEWAKE#): now also R28.2
- new net: FL2.3, J2.5 (D+)
- new net: FL2.4, J2.3 (D-)
- new net: FL1.3, J2.4 (D-)
- new net: FL1.4, J2.6 (D+)
- new net +3.3V: D3.2 (A), F1.2
Other:
- note added: "DOWNSTREAM PORT1 / PORT2"
- note added: "PCIe M2 Key M+B"
- company: 3mdeb Sp. z o.o -> 3mdeb Sp. z o.o    Jakub Sobota
- moved on the sheet: J1, J2

Commit message: Placed additional information to board schematics
Signed-off-by: Jakub Sobota <jakub.sobota@3mdeb.com>
Other:
- note added: "-MIN VIA PAD SIZE 20mils -MIN spacing between trace and pad is 5mils -MIN spacing between VIA and pad is 5mils -MIN width of trace is 4mils"
- note added: "-USB_DP/M must be 90-ohm differential (+/-15%) -PCIE_TXP/N must be 100-ohms differential (+/-10%) -PCIE_RXP/N must be 100-ohms differential (+/-10%) -PCIE_REFCLKP/N must be 100-ohms differential (+/-10%)"
- note added: "-USB_DP/M within 25mils -PCIE_TXP/N within 5mils -PCIE_RXP/N within 5mils -PCIE_REFCLKP/N within 25mils"
- note added: "IMPEDANCE REQUIREMENTS:"
- note added: "LENGTH MATCHING REQUIREMENTS:"
- note added: "VIA AND TRACE REQUIREMENTS:"
- moved on the sheet: FL1, FL2, J2

Commit message: Updated PCB Design
Signed-off-by: Jakub Sobota <jakub.sobota@3mdeb.com>
Connections:
- net DM2: now also FL1.4; no longer FL1.2
- net DP2: now also FL1.3; no longer FL1.1
- net at J2.4 (D-): now also FL1.1; no longer FL1.3
- net at J2.6 (D+): now also FL1.2; no longer FL1.4
