File: Kicad-Files/PCI2USB.kicad_sch (KiCad schematic)
At the start: 15 parts, among them J2 USB_9PIN_Internal

Commit message: Cleaned custom libraries, fixed footprint and 3d models
Signed-off-by: Jakub Sobota <jakub.sobota@3mdeb.com>
Parts:
- removed D3: 4V/5A, Diode_SMD:D_SOD-323_HandSoldering, symbol Diode:PTVS5V0Z1USK
- removed FL1, FL2: 90 Ohm, Filters:MCZ1210AH_CP, symbol Filter:Choke_CommonMode_PulseElectronics_PH9455x405NL
- removed J1: ~, M2_Edge_connector:M.2_KEY_M_B, symbol M2_Edge_connector:M.2_Key_M_B
- added D3: PJSD03TS-AU, PJSD0XTS-AU:PJSD0XTS-AU, symbol PJSD0XTS-AU:PJSD03TS-AU
- added FL1, FL2: Choke_CommonMode_PulseElectronics_PH9455x105NL, MCZ1210AH900L2TA0G:MCZ1210AH201L2TA0G, symbol MCZ1210AH900L2TA0G:MCZ1210AH900L2TA0G
- added J1: ~, Connectors:M.2_KEY_M_B, symbol Connectors:M.2_Key_M_B
Connections:
- net +3.3V: now also C17.1, C18.1, C19.1, C20.1, C21.1, F1.1, D3.1 (K), J1.2 (3.3V), J1.4 (3.3V), J1.70 (3.3V), J1.72 (3.3V), J1.74 (3.3V)
- net DM1: now also FL2.1
- net DM2: now also FL1.2
- net DP1: now also FL2.2
- net DP2: now also FL1.1
- net DS1_VBUS: now also J2.8 (GND); no longer J2.1 (5V)
- net DS2_VBUS: now also J2.7 (GND); no longer J2.2 (5V)
- net GND: now also J2.1 (5V), J2.2 (5V), D3.2 (A), J1.27 (GND), J1.3 (GND), J1.33 (GND), J1.39 (GND), J1.45 (GND), J1.51 (GND), J1.57 (GND), J1.71 (GND), J1.73 (GND); no longer J2.7 (GND), J2.8 (GND)
- net PCIE_REFCLKN: now also J1.53 (REFCLKn)
- net PCIE_REFCLKP: now also J1.55 (REFCLKp)
- net PCIE_RXN: now also J1.47 (PETn0/SATA-A-)
- net PCIE_RXP: now also J1.49 (PETp0/SATA-A+)
- net PERSTZ: now also J1.50 (PERST#)
- net at C14.1: now also J1.41 (PERn0/SATA-B+)
- net at J2.4 (D-): now also FL2.3
- net at J2.6 (D+): now also FL2.4
- net at J2.5 (D+): now also FL1.3
- net at J2.3 (D-): now also FL1.4
- net at C15.1: now also J1.43 (PERp0/SATA-B-)
- net at R28.2: now also J1.54 (PEWAKE#)
Other:
- moved on the sheet: C14, C15, C16, R28

Commit message: Redesigned PCB compliant with PCI and SS USB standards
Signed-off-by: Jakub Sobota <jakub.sobota@3mdeb.com>
Parts:
- removed FL2: Choke_CommonMode_PulseElectronics_PH9455x105NL, MCZ1210AH900L2TA0G:MCZ1210AH201L2TA0G, symbol MCZ1210AH900L2TA0G:MCZ1210AH900L2TA0G
- added FL1: 90 Ohm 160mA, MCZ1210AH900L2TA0G:MCZ1210AH201L2TA0G, symbol MCZ1210AH900L2TA0G:MCZ1210AH900L2TA0G
- C14, C15: footprint Capacitor_SMD:C_0402_1005Metric_Pad0.74x0.62mm_HandSolder -> Capacitor_SMD:C_0402_1005Metric
- D3: value PJSD03TS-AU -> 4V/6.5V/5A
- FL2: renamed from FL1; value Choke_CommonMode_PulseElectronics_PH9455x105NL -> 90 Ohm 160mA
- J1: value ~ -> M.2 Edge Connector
Connections:
- net +3.3V: no longer C17.1, C18.1, C19.1, C20.1, C21.1, F1.1, J1.2 (3.3V), J1.4 (3.3V), J1.70 (3.3V), J1.72 (3.3V), J1.74 (3.3V)
- net DM1: now also FL1.2
- net DM2: now also FL2.1; no longer FL2.2
- net DP1: now also FL1.1
- net DP2: now also FL2.2; no longer FL2.1
- net DS1_VBUS: now also J2.7 (GND); no longer J2.8 (GND)
- net DS2_VBUS: now also J2.8 (GND); no longer J2.7 (GND)
- net at J2.4 (D-): now also FL1.3
- net at J2.6 (D+): now also FL1.4
- new net: C17.1, C18.1, C19.1, C20.1, C21.1, F1.1, J1.2 (3.3V), J1.4 (3.3V), J1.70 (3.3V), J1.72 (3.3V), J1.74 (3.3V)

Commit message: Fixed reversed 9 pin connector
Signed-off-by: Jakub Sobota <jakub.sobota@3mdeb.com>
Connections:
- net DS1_VBUS: now also J2.2 (5V); no longer J2.7 (GND)
- net DS2_VBUS: now also J2.1 (5V); no longer J2.8 (GND)
- net GND: now also J2.7 (GND), J2.8 (GND); no longer J2.1 (5V), J2.2 (5V)
Changed lines of the file:
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@@
-	(wire
-		(pts
-			(xy 236.22 68.58) (xy 251.46 68.58)
-		)
-		(stroke
-			(width 0)
-			(type default)
-		)
-	)
 	(wire
 		(pts
@@
 	(wire
 		(pts
-			(xy 213.36 68.58) (xy 195.58 68.58)
-		)
-		(stroke
-			(width 0)
-			(type default)
-		)
-	)
-	(wire
-		(pts
 			(xy 123.19 81.28) (xy 129.54 81.28)
 		)
@@
 	(wire
 		(pts
+			(xy 100.33 124.46) (xy 115.57 124.46)
+		)
+		(stroke
+			(width 0)
+			(type default)
+		)
+	)
+	(wire
+		(pts
+			(xy 113.03 81.28) (xy 118.11 81.28)
+		)
+		(stroke
+			(width 0)
+			(type default)
+		)
+	)
+	(wire
+		(pts
+			(xy 52.07 111.76) (xy 64.77 111.76)
+		)
+		(stroke
+			(width 0)
+			(type default)
+		)
+	)
+	(wire
+		(pts
+			(xy 44.45 116.84) (xy 64.77 116.84)
+		)
+		(stroke
+			(width 0)
+			(type default)
+		)
+	)
+	(wire
+		(pts
+			(xy 113.03 59.69) (xy 116.84 59.69)
+		)
+		(stroke
+			(width 0)
+			(type default)
+		)
+	)
+	(wire
+		(pts
+			(xy 123.19 127) (xy 123.19 124.46)
+		)
+		(stroke
+			(width 0)
+			(type default)
+		)
+	)
+	(wire
+		(pts
+			(xy 209.55 52.07) (xy 209.55 55.88)
+		)
+		(stroke
+			(width 0)
+			(type default)
+		)
+	)
+	(wire
+		(pts
+			(xy 59.69 91.44) (xy 59.69 99.06)
+		)
+		(stroke
+			(width 0)
+			(type default)
+		)
+	)
+	(wire
+		(pts
+			(xy 52.07 113.03) (xy 52.07 111.76)
+		)
+		(stroke
+			(width 0)
+			(type default)
+		)
+	)
+	(wire
+		(pts
+			(xy 215.9 60.96) (xy 212.09 60.96)
+		)
+		(stroke
+			(width 0)
+			(type default)
+		)
+	)
+	(wire
+		(pts
+			(xy 113.03 88.9) (xy 118.11 88.9)
+		)
+		(stroke
+			(width 0)
+			(type default)
+		)
+	)
+	(wire
+		(pts
+			(xy 209.55 55.88) (xy 215.9 55.88)
+		)
+		(stroke
+			(width 0)
+			(type default)
+		)
+	)
+	(wire
+		(pts
+			(xy 195.58 52.07) (xy 209.55 52.07)
+		)
+		(stroke
+			(width 0)
+			(type default)
+		)
+	)
+	(wire
+		(pts
+			(xy 59.69 121.92) (xy 64.77 121.92)
+		)
+		(stroke
+			(width 0)
+			(type default)
+		)
+	)
+	(wire
+		(pts
+			(xy 48.26 124.46) (xy 64.77 124.46)
+		)
+		(stroke
+			(width 0)
+			(type default)
+		)
+	)
+	(wire
+		(pts
 			(xy 238.76 52.07) (xy 238.76 55.88)
 		)
@@
 	(wire
 		(pts
-			(xy 100.33 124.46) (xy 115.57 124.46)
-		)
-		(stroke
-			(width 0)
-			(type default)
-		)
-	)
-	(wire
-		(pts
-			(xy 113.03 81.28) (xy 118.11 81.28)
-		)
-		(stroke
-			(width 0)
-			(type default)
-		)
-	)
-	(wire
-		(pts
-			(xy 52.07 111.76) (xy 64.77 111.76)
-		)
-		(stroke
-			(width 0)
-			(type default)
-		)
-	)
-	(wire
-		(pts
-			(xy 44.45 116.84) (xy 64.77 116.84)
-		)
-		(stroke
-			(width 0)
-			(type default)
-		)
-	)
-	(wire
-		(pts
-			(xy 113.03 59.69) (xy 116.84 59.69)
-		)
-		(stroke
-			(width 0)
-			(type default)
-		)
-	)
-	(wire
-		(pts
-			(xy 123.19 127) (xy 123.19 124.46)
-		)
-		(stroke
-			(width 0)
-			(type default)
-		)
-	)
-	(wire
-		(pts
-			(xy 59.69 91.44) (xy 59.69 99.06)
-		)
-		(stroke
-			(width 0)
-			(type default)
-		)
-	)
-	(wire
-		(pts
-			(xy 52.07 113.03) (xy 52.07 111.76)
-		)
-		(stroke
-			(width 0)
-			(type default)
-		)
-	)
-	(wire
-		(pts
-			(xy 215.9 60.96) (xy 212.09 60.96)
-		)
-		(stroke
-			(width 0)
-			(type default)
-		)
-	)
-	(wire
-		(pts
-			(xy 113.03 88.9) (xy 118.11 88.9)
-		)
-		(stroke
-			(width 0)
-			(type default)
-		)
-	)
-	(wire
-		(pts
-			(xy 209.55 55.88) (xy 215.9 55.88)
-		)
-		(stroke
-			(width 0)
-			(type default)
-		)
-	)
-	(wire
-		(pts
-			(xy 59.69 121.92) (xy 64.77 121.92)
-		)
-		(stroke
-			(width 0)
-			(type default)
-		)
-	)
-	(wire
-		(pts
-			(xy 48.26 124.46) (xy 64.77 124.46)
-		)
-		(stroke
-			(width 0)
-			(type default)
-		)
-	)
-	(wire
-		(pts
 			(xy 118.11 77.47) (xy 113.03 77.47)
 		)
@@
 	(wire
 		(pts
-			(xy 209.55 52.07) (xy 209.55 55.88)
+			(xy 252.73 52.07) (xy 238.76 52.07)
 		)
 		(stroke
@@
 	(global_label "DS1_VBUS"
 		(shape input)
-		(at 195.58 68.58 180)
+		(at 252.73 52.07 0)
 		(fields_autoplaced yes)
 		(effects
@@
 				(size 1.27 1.27)
 			)
-			(justify right)
+			(justify left)
 		)
 		(property "Intersheetrefs" "${INTERSHEET_REFS}"
-			(at 183.0396 68.58 0)
-			(effects
-				(font
-					(size 1.27 1.27)
-				)
-				(justify right)
+			(at 265.2704 52.07 0)
+			(effects
+				(font
+					(size 1.27 1.27)
+				)
+				(justify left)
 			)
 		)
@@
 	(global_label "DS2_VBUS"
 		(shape input)
-		(at 251.46 68.58 0)
+		(at 195.58 52.07 180)
 		(fields_autoplaced yes)
 		(effects
@@
 				(size 1.27 1.27)
 			)
-			(justify left)
+			(justify right)
 		)
 		(property "Intersheetrefs" "${INTERSHEET_REFS}"
-			(at 264.0004 68.58 0)
-			(effects
-				(font
-					(size 1.27 1.27)
-				)
-				(justify left)
+			(at 183.0396 52.07 0)
+			(effects
+				(font
+					(size 1.27 1.27)
+				)
+				(justify right)
 			)
 		)
@@
 	(symbol
 		(lib_id "power:GND")
-		(at 238.76 52.07 180)
+		(at 236.22 68.58 0)
 		(unit 1)
 		(exclude_from_sim no)
@@
 		(fields_autoplaced yes)
 		(property "Reference" "#PWR021"
-			(at 238.76 45.72 0)
+			(at 236.22 74.93 0)
 			(effects
 				(font
@@
 		)
 		(property "Value" "GND"
-			(at 238.76 46.99 0)
+			(at 236.22 73.66 0)
 			(effects
 				(font
@@
 		)
 		(property "Footprint" ""
-			(at 238.76 52.07 0)
+			(at 236.22 68.58 0)
 			(effects
 				(font
@@
 		)
 		(property "Datasheet" ""
-			(at 238.76 52.07 0)
+			(at 236.22 68.58 0)
 			(effects
 				(font
@@
 		)
 		(property "Description" "Power symbol creates a global label with name \"GND\" , ground"
-			(at 238.76 52.07 0)
+			(at 236.22 68.58 0)
 			(effects
 				(font
@@
 		(on_board yes)
 		(dnp no)
-		(fields_autoplaced yes)
 		(property "Reference" "FL2"
-			(at 197.739 52.07 0)
+			(at 197.866 55.626 0)
 			(effects
 				(font
@@
 	(symbol
 		(lib_id "power:GND")
-		(at 209.55 52.07 180)
+		(at 213.36 68.58 0)
 		(unit 1)
 		(exclude_from_sim no)
@@
 		(fields_autoplaced yes)
 		(property "Reference" "#PWR019"
-			(at 209.55 45.72 0)
+			(at 213.36 74.93 0)
 			(effects
 				(font
@@
 		)
 		(property "Value" "GND"
-			(at 209.55 46.99 0)
+			(at 213.36 73.66 0)
 			(effects
 				(font
@@
 		)
 		(property "Footprint" ""
-			(at 209.55 52.07 0)
+			(at 213.36 68.58 0)
 			(effects
 				(font
@@
 		)
 		(property "Datasheet" ""
-			(at 209.55 52.07 0)
+			(at 213.36 68.58 0)
 			(effects
 				(font
@@
 		)
 		(property "Description" "Power symbol creates a global label with name \"GND\" , ground"
-			(at 209.55 52.07 0)
-			(effects
-				(font
+			(at 213.36 68.58 0)
+			(effects
+				(font

Commit message: fixed pdf schematics, removed temporary files
Signed-off-by: Jakub Sobota <jakub.sobota@3mdeb.com>
Changed lines of the file:
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@@
 	(title_block
 		(title "PCI2USB")
-		(date "2025-11-17")
+		(date "2025-12-08")
 		(rev "1.0.0")
 		(company "3mdeb Sp. z o.o    Jakub Sobota")
@@
 	)
 	(rectangle
-		(start 26.67 40.64)
+		(start 25.4 40.64)
 		(end 142.24 190.5)
 		(stroke
