File: Kicad-Files/TUSB7320 Power.kicad_sch (KiCad schematic)
At the start: 13 parts, among them U3 TPS74401

Commit message: Created schematics for TUSB7320 USB Controller
Signed-off-by: Jakub Sobota <jakub.sobota@3mdeb.com>
Changed lines of the file:
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@@
+		)
+	)
+	(global_label "GRSTZ"
+		(shape input)
+		(at 195.58 85.09 0)
+		(fields_autoplaced yes)
+		(effects
+			(font
+				(size 1.27 1.27)
+			)
+			(justify left)
+		)
+		(property "Intersheetrefs" "${INTERSHEET_REFS}"
+			(at 204.4918 85.09 0)
+			(effects
+				(font
+					(size 1.27 1.27)
+				)
+				(justify left)
+			)
 		)
 	)
@@
 					(unit 1)
 				)
-			)
-		)
-	)
-	(symbol
-		(lib_id "power:LINE")
-		(at 195.58 85.09 270)
-		(unit 1)
-		(exclude_from_sim no)
-		(in_bom yes)
-		(on_board yes)
-		(dnp no)
-		(fields_autoplaced yes)
-		(property "Reference" "#PWR024"
-			(at 191.77 85.09 0)
-			(effects
-				(font
-					(size 1.27 1.27)
-				)
-				(hide yes)
-			)
-		)
-		(property "Value" "GRSTZ"
-			(at 199.39 85.0899 90)
-			(effects
-				(font
-					(size 1.27 1.27)
-				)
-				(justify left)
-			)
-		)
-		(property "Footprint" ""
-			(at 195.58 85.09 0)
-			(effects
-				(font
-					(size 1.27 1.27)
-				)
-				(hide yes)
-			)
-		)
-		(property "Datasheet" ""
-			(at 195.58 85.09 0)
-			(effects
-				(font
-					(size 1.27 1.27)
-				)
-				(hide yes)
-			)
-		)
-		(property "Description" "Power symbol creates a global label with name \"LINE\""
-			(at 195.58 85.09 0)
-			(effects
-				(font
-					(size 1.27 1.27)
-				)
-				(hide yes)
-			)
-		)
-		(pin "1"
-		)
-		(instances
-			(project ""
-				(path "/513f496d-ec7a-4c1e-814f-35a10c718f03/641a18fa-9239-44e7-9711-1a374441a862"
-					(reference "#PWR024")
-					(unit 1)
-				)

Commit message: Complete Schematics and BOM
Signed-off-by: Jakub Sobota <jakub.sobota@3mdeb.com>
Parts:
- added C22, C25, C28, C31, C37, C40, C43, C46, C49, C57: 0.01 μF, Capacitor_SMD:C_0402_1005Metric_Pad0.74x0.62mm_HandSolder, symbol Device:C_Small
- added C23, C24, C26, C27, C29, C30, C32, C33, C38, C39, C41, C42, C44, C45, C47, C48, C50, C51, C52, C53, C54, C55: 0.1 μF, Capacitor_SMD:C_0402_1005Metric_Pad0.74x0.62mm_HandSolder, symbol Device:C_Small
- added C34, C56: 22 μF, Capacitor_SMD:C_0805_2012Metric_Pad1.18x1.45mm_HandSolder, symbol Device:C_Small
- added FB1: 220 Ohm, Inductor_SMD:L_0603_1608Metric_Pad1.05x0.95mm_HandSolder, symbol Device:FerriteBead_Small
Connections:
- net +1.1V: now also C22.1, C23.1, C24.1, C25.1, C26.1, C27.1, C28.1, C29.1, C30.1, C31.1, C32.1, C33.1, C34.1, C37.1, C38.1, C39.1, C40.1, C41.1, C42.1, C43.1, C44.1
- net +3.3V: now also C51.1, C52.1, C53.1, C54.1, C55.1, FB1.2
- net GND: now also C22.2, C23.2, C24.2, C25.2, C26.2, C27.2, C28.2, C29.2, C30.2, C31.2, C32.2, C33.2, C34.2, C37.2, C38.2, C39.2, C40.2, C41.2, C42.2, C43.2, C44.2, C45.2, C46.2, C47.2, C48.2, C49.2, C50.2, C51.2, C52.2, C53.2, C54.2, C55.2, C56.2, C57.2
- new net VDDA_3P3: C45.1, C46.1, C47.1, C48.1, C49.1, C50.1, C56.1, C57.1, FB1.1
Other:
- note added: "1.1V LINE CAPACITORS"
- note added: "1.1V REGULATOR"
- note added: "3.3V LINE CAPACITORS"
- company: 3mdeb Sp. z o.o -> 3mdeb Sp. z o.o    Jakub Sobota
- moved on the sheet: C4, C5, C6, C7, C8, D5, F3, R5, R6, R7, R8, R9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

Commit message: Placed additional information to board schematics
Signed-off-by: Jakub Sobota <jakub.sobota@3mdeb.com>
Changed lines of the file:
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@@
 	)
 	(rectangle
-		(start 41.91 97.79)
+		(start 44.45 97.79)
 		(end 203.2 142.24)
 		(stroke
@@
 	(text "1.1V LINE CAPACITORS"
 		(exclude_from_sim no)
-		(at 60.452 97.028 0)
+		(at 61.976 95.758 0)
 		(effects
 			(font

Commit message: Cleaned custom libraries, fixed footprint and 3d models
Signed-off-by: Jakub Sobota <jakub.sobota@3mdeb.com>
Parts:
- removed U3: TPS74401, Package_DFN_QFN:Texas_RGW0020A_VQFN-20-1EP_5x5mm_P0.65mm_EP3.15x3.15mm_ThermalVias, symbol DC-DC Converter:TPS74401_VQFN
- added U2: TPS74401, TPS74401:TPS74401RGWRM3, symbol TPS74401:TPS74401RGWRM3
Connections:
- net +1.1V: now also U2.1 (OUT), U2.18 (OUT), U2.19 (OUT), U2.20 (OUT)
- net GND: now also U2.12 (GND), U2.13 (NC), U2.14 (NC), U2.17 (NC), U2.21 (PAD), U2.3 (NC), U2.4 (NC)
- net GRSTZ: now also U2.9 (PG)
- net at C4.1, D5.2 (A), F3.2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: now also U2.10 (BIAS), U2.5 (IN), U2.6 (IN), U2.7 (IN), U2.8 (IN)
- net at C8.2, R8.2: now also U2.11 (EN)
- net at C5.1: now also U2.15 (SS)
- net at R5.2, R6.2: now also U2.16 (FB)
Changed lines of the file:
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@@
 	(wire
 		(pts
-			(xy 109.22 38.1) (xy 109.22 44.45)
-		)
-		(stroke
-			(width 0)
-			(type default)
-		)
-	)
-	(wire
-		(pts
 			(xy 50.8 177.8) (xy 60.96 177.8)
 		)
@@
 	(wire
 		(pts
+			(xy 109.22 38.1) (xy 109.22 44.45)
+		)
+		(stroke
+			(width 0)
+			(type default)
+		)
+	)
+	(wire
+		(pts
 			(xy 165.1 110.49) (xy 175.26 110.49)
 		)
@@
 	)
 	(symbol
-		(lib_id "DC-DC Converter:TPS74401_VQFN")
-		(at 124.46 54.61 0)
-		(unit 1)
-		(exclude_from_sim no)
-		(in_bom yes)
-		(on_board yes)
-		(dnp no)
-		(fields_autoplaced yes)
-		(property "Reference" "U3"
-			(at 130.175 38.1 0)
-			(effects
-				(font
-					(size 1.27 1.27)
-				)
-			)
-		)
-		(property "Value" "TPS74401"
-			(at 130.175 40.64 0)
-			(effects
-				(font
-					(size 1.27 1.27)
-				)
-			)
-		)
-		(property "Footprint" "Package_DFN_QFN:Texas_RGW0020A_VQFN-20-1EP_5x5mm_P0.65mm_EP3.15x3.15mm_ThermalVias"
-			(at 144.78 69.85 0)
-			(effects
-				(font
-					(size 1.27 1.27)
-				)
-				(hide yes)
-			)
-		)
-		(property "Datasheet" "https://www.ti.com/lit/gpn/tps74401"
-			(at 129.54 35.56 0)
-			(effects
-				(font
-					(size 1.27 1.27)
-				)
-				(hide yes)
-			)
-		)
-		(property "Description" "0.8 to 3.6V adjustable, 3.0-A, Ultra-LDO with Programmable Soft-Start"
-			(at 140.716 75.438 0)
-			(effects
-				(font
-					(size 1.27 1.27)
-				)
-				(hide yes)
-			)
-		)
-		(pin "9"
-		)
-		(pin "17"
-		)
-		(pin "18"
-		)
-		(pin "10"
-		)
-		(pin "12"
-		)
-		(pin "7"
-		)
-		(pin "14"
-		)
-		(pin "16"
-		)
-		(pin "19"
-		)
-		(pin "15"
-		)
-		(pin "1"
-		)
-		(pin "8"
-		)
-		(pin "21"
-		)
-		(pin "11"
-		)
-		(pin "3"
-		)
-		(pin "6"
-		)
-		(pin "20"
-		)
-		(pin "2"
-		)
-		(pin "4"
-		)
-		(pin "13"
-		)
-		(pin "5"
-		)
-		(instances
-			(project ""
-				(path "/513f496d-ec7a-4c1e-814f-35a10c718f03/641a18fa-9239-44e7-9711-1a374441a862"
-					(reference "U3")
-					(unit 1)
-				)
-			)
-		)
-	)
-	(symbol
 		(lib_id "Device:C_Small")
 		(at 92.71 128.27 0)
@@
 	)
 	(symbol
-		(lib_id "power:+3.3V")
-		(at 62.23 52.07 90)
-		(unit 1)
-		(exclude_from_sim no)
-		(in_bom yes)
-		(on_board yes)
-		(dnp no)
-		(fields_autoplaced yes)
-		(property "Reference" "#PWR011"
-			(at 66.04 52.07 0)
-			(effects
-				(font
-					(size 1.27 1.27)
-				)
-				(hide yes)
-			)
-		)
-		(property "Value" "+3.3V"
-			(at 58.42 52.0699 90)
-			(effects
-				(font
-					(size 1.27 1.27)
-				)
-				(justify left)
-			)
-		)
-		(property "Footprint" ""
-			(at 62.23 52.07 0)
-			(effects
-				(font
-					(size 1.27 1.27)
-				)
-				(hide yes)
-			)
-		)
-		(property "Datasheet" ""
-			(at 62.23 52.07 0)
-			(effects
-				(font
-					(size 1.27 1.27)
-				)
-				(hide yes)
-			)
-		)
-		(property "Description" "Power symbol creates a global label with name \"+3.3V\""
-			(at 62.23 52.07 0)
-			(effects
-				(font
-					(size 1.27 1.27)
-				)
-				(hide yes)
-			)
-		)
-		(pin "1"
-		)
-		(instances
-			(project ""
-				(path "/513f496d-ec7a-4c1e-814f-35a10c718f03/641a18fa-9239-44e7-9711-1a374441a862"
-					(reference "#PWR011")
-					(unit 1)
-				)
-			)
-		)
-	)
-	(symbol
 		(lib_id "Device:C_Small")
 		(at 165.1 113.03 0)
@@
 	)
 	(symbol
+		(lib_id "TPS74401:TPS74401RGWRM3")
+		(at 124.46 54.61 0)
+		(unit 1)
+		(exclude_from_sim no)
+		(in_bom yes)
+		(on_board yes)
+		(dnp no)
+		(fields_autoplaced yes)
+		(property "Reference" "U2"
+			(at 130.175 38.1 0)
+			(effects
+				(font
+					(size 1.27 1.27)
+				)
+			)
+		)
+		(property "Value" "TPS74401"
+			(at 130.175 40.64 0)
+			(effects
+				(font
+					(size 1.27 1.27)
+				)
+			)
+		)
+		(property "Footprint" "TPS74401:TPS74401RGWRM3"
+			(at 139.7 80.772 0)
+			(effects
+				(font
+					(size 1.27 1.27)
+				)
+				(hide yes)
+			)
+		)
+		(property "Datasheet" "https://www.ti.com/lit/gpn/tps74401"
+			(at 129.54 35.56 0)
+			(effects
+				(font
+					(size 1.27 1.27)
+				)
+				(hide yes)
+			)
+		)
+		(property "Description" "0.8 to 3.6V adjustable, 3.0-A, Ultra-LDO with Programmable Soft-Start"
+			(at 135.636 86.36 0)
+			(effects
+				(font
+					(size 1.27 1.27)
+				)
+				(hide yes)
+			)
+		)
+		(pin "14"
+		)
+		(pin "12"
+		)
+		(pin "9"
+		)
+		(pin "11"
+		)
+		(pin "2"
+		)
+		(pin "21"
+		)
+		(pin "4"
+		)
+		(pin "3"
+		)
+		(pin "20"
+		)
+		(pin "1"
+		)
+		(pin "15"
+		)
+		(pin "10"
+		)
+		(pin "8"
+		)
+		(pin "7"
+		)
+		(pin "6"
+		)
+		(pin "19"
+		)
+		(pin "16"
+		)
+		(pin "5"
+		)
+		(pin "17"
+		)
+		(pin "13"
+		)
+		(pin "18"
+		)
+		(instances
+			(project ""
+				(path "/513f496d-ec7a-4c1e-814f-35a10c718f03/641a18fa-9239-44e7-9711-1a374441a862"
+					(reference "U2")
+					(unit 1)
+				)
+			)
+		)
+	)
+	(symbol
 		(lib_id "power:GND")
 		(at 171.45 38.1 0)
@@
 					(unit 1)
 				)
+			)
+		)
+	)
+	(symbol
+		(lib_id "power:+3.3V")
+		(at 62.23 52.07 90)
+		(unit 1)
+		(exclude_from_sim no)
+		(in_bom yes)
+		(on_board yes)
+		(dnp no)
+		(property "Reference" "#PWR052"
+			(at 66.04 52.07 0)
+			(effects
+				(font
+					(size 1.27 1.27)
+				)
+				(hide yes)
+			)
+		)
+		(property "Value" "+3.3V"
+			(at 57.15 52.07 0)
+			(effects
+				(font
+					(size 1.27 1.27)
+				)
+			)
+		)
+		(property "Footprint" ""
+			(at 62.23 52.07 0)
+			(effects
+				(font
+					(size 1.27 1.27)
+				)
+				(hide yes)
+			)
+		)
+		(property "Datasheet" ""
+			(at 62.23 52.07 0)
+			(effects
+				(font
+					(size 1.27 1.27)
+				)
+				(hide yes)
+			)
+		)
+		(property "Description" "Power symbol creates a global label with name \"+3.3V\""
+			(at 62.23 52.07 0)
+			(effects
+				(font
+					(size 1.27 1.27)
+				)
+				(hide yes)
+			)
+		)
+		(pin "1"
+		)
+		(instances
+			(project ""
+				(path "/513f496d-ec7a-4c1e-814f-35a10c718f03/641a18fa-9239-44e7-9711-1a374441a862"
+					(reference "#PWR052")
+					(unit 1)
+				)

Commit message: Redesigned PCB compliant with PCI and SS USB standards
Signed-off-by: Jakub Sobota <jakub.sobota@3mdeb.com>
Parts:
- removed D5: LED, LED_SMD:LED_0603_1608Metric_Pad1.05x0.95mm_HandSolder, symbol Device:LED
- removed R9: 330 Ohm, Resistor_SMD:R_0402_1005Metric_Pad0.72x0.64mm_HandSolder, symbol Device:R_Small_US
- renumbered U2 to U3
Other:
- moved on the sheet: F3

Commit message: Updated all SMD footprints to not hand soldered versions
Signed-off-by: Jakub Sobota <jakub.sobota@3mdeb.com>
Parts:
- C22, C23, C24, C25, C26, C27, C28, C29, C30, C31, C32, C33, C37, C38, C39, C40, C41, C42, C43, C44, C45, C46, C47, C48, C49, C50, C51, C52, C53, C54, C55, C57, C6, C8: footprint Capacitor_SMD:C_0402_1005Metric_Pad0.74x0.62mm_HandSolder -> Capacitor_SMD:C_0402_1005Metric
- C34, C4, C56, C7: footprint Capacitor_SMD:C_0805_2012Metric_Pad1.18x1.45mm_HandSolder -> Capacitor_SMD:C_0805_2012Metric
- F3: footprint Fuse:Fuse_0603_1608Metric_Pad1.05x0.95mm_HandSolder -> Fuse:Fuse_0603_1608Metric
- FB1: footprint Inductor_SMD:L_0603_1608Metric_Pad1.05x0.95mm_HandSolder -> Inductor_SMD:L_0603_1608Metric
- R5, R6, R7, R8: footprint Resistor_SMD:R_0402_1005Metric_Pad0.72x0.64mm_HandSolder -> Resistor_SMD:R_0402_1005Metric
