File: Kicad-Files/USB Power.kicad_sch (KiCad schematic)
At the start: 27 parts, among them U1 TPS61023DRLR, U2 TPS2560DRC

Commit message: Redesigned schematic and board REV 2.0
Parts:
- removed C11: 0.1 μF, Capacitor_SMD:C_0402_1005Metric, symbol Device:C_Small
- removed C12, C13: 150uF, Capacitor_SMD:CP_Elec_6.3x5.9, symbol Device:C_Polarized_Small_US
- removed C2: 22 μF, Capacitor_SMD:C_0805_2012Metric, symbol Device:C_Small
- removed D2: 6V/9V/5A, PJSD0XTS-AU:PJSD0XTS-AU, symbol PJSD0XTS-AU:PJSD03TS-AU
- removed F2: 5A, Fuse:Fuse_0603_1608Metric, symbol Device:Fuse_Small
- removed R15, R16: NOPOP, Resistor_SMD:R_0402_1005Metric_Pad0.72x0.64mm_HandSolder, symbol Device:R_US
- removed R29: 100 KOhm, Resistor_SMD:R_0402_1005Metric, symbol Device:R_US
- added C13, C15, C9: 100u_6.3V, Capacitor_SMD:C_1206_3216Metric, symbol Device:C_Small
- added C14: 0.1u, Capacitor_SMD:C_0402_1005Metric, symbol Device:C_Small
- added D3, D4: 6V/9V/5A, PJSD0XTS-AU:PJSD0XTS-AU, symbol PJSD0XTS-AU:PJSD03TS-AU
- C10: renamed from C9; value 0.1 μF -> 0.1u
- C11: renamed from C3; value 22 μF -> 22u
- C12: renamed from C10; value 0.1 μF -> 0.1u
- C8: renamed from C1; value 22 μF -> 22u
- D2: renamed from D4; value LED -> RED
- D5: renamed from D6; value LED -> GRN
- D6: renamed from D7; value LED -> GRN
- L3: renamed from L1; value 1 μH -> 1u
- R10: renamed from R19; value 10 KOhm -> 10K
- R11: renamed from R4; value 1.5 KOhm -> 1.5K
- R12: renamed from R20; value 680 Ohm -> 680R
- R13: renamed from R21; value 680 Ohm -> 680R
- R6: renamed from R2; value 100 KOhm -> 100K_1%
- R7: renamed from R1; value 732 KOhm -> 732K_1%; footprint Resistor_SMD:R_0603_1608Metric -> Resistor_SMD:R_0402_1005Metric
- R8: renamed from R17; value 30.9 KOhm -> 30.9K_1%
- R9: renamed from R18; value 10 KOhm -> 10K
- renumbered U1 to U3, U2 to U4
Connections:
- net +3.3V: now also U3.2 (EN)
- net +5V: now also C11.2, D2.2 (A), R7.2, U3.6 (VOUT), C9.1
- net DS1_VBUS: now also D6.2 (A), U4.8 (OUT2), C14.1, C15.1, D4.1 (K); no longer C12.1, D5.2 (A), U4.9 (OUT1)
- net DS2_VBUS: now also C12.1, D5.2 (A), U4.9 (OUT1), C13.1, D3.1 (K); no longer D6.2 (A), U4.8 (OUT2)
- net GND: now also C13.2, C14.2, C15.2, C9.2, D3.2 (A), D4.2 (A)
- net OVERCUR1Z: now also R10.1, U4.6 (~{FAULT2}); no longer R9.1, U4.10 (~{FAULT1})
- net OVERCUR2Z: now also R9.1, U4.10 (~{FAULT1}); no longer R10.1, U4.6 (~{FAULT2})
- net PWRON1Z: now also U4.5 (EN2); no longer U4.4 (EN1)
- net PWRON2Z: now also U4.4 (EN1); no longer U4.5 (EN2)
Other:
- note added: "100uF CAPS: https://www.lcsc.com/product-detail/C15008.html"
- company: 3mdeb Sp. z o.o    Jakub Sobota -> 3mdeb Sp. z o.o    Dominik Baroński
- title: PCI2USB -> PCI2USB USB power
- moved on the sheet: C10, C11, C12, C8, D2, D5, D6, L3, R10, R11, R12, R13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
