File: Kicad-Files/USBController.kicad_sch (KiCad schematic)
At the start: 15 parts, among them U2 TUSB7320, Y1 Crystal

Commit message: Complete Schematics and BOM
Signed-off-by: Jakub Sobota <jakub.sobota@3mdeb.com>
Parts:
- removed Y1: Crystal, symbol Device:Crystal
- added Y2: 48 MHz, Crystal:Crystal_SMD_Abracon_ABM3B-4Pin_5.0x3.2mm, symbol Device:Crystal_GND24_Small
- C35, C36: footprint (none) -> Capacitor_SMD:C_0402_1005Metric_Pad0.74x0.62mm_HandSolder
- R10: value 9 KOhm -> 9.09 KOhm; footprint (none) -> Resistor_SMD:R_0402_1005Metric_Pad0.72x0.64mm_HandSolder
- R11, R12, R13, R14, R22, R23, R26, R27: footprint (none) -> Resistor_SMD:R_0402_1005Metric_Pad0.72x0.64mm_HandSolder
- R24, R25: value 1 Ohm -> 0 Ohm; footprint (none) -> LED_SMD:LED_0402_1005Metric_Pad0.77x0.64mm_HandSolder
Connections:
- net GND: now also Y2.2, Y2.4
- net at U2.A49 (GPIO0): now also R14.2; no longer R13.2
- net at C35.2, R27.2, U2.A23 (XI): now also Y2.3
- net at C36.2, R27.1, U2.A22 (XO): now also Y2.1
- net at U2.B46 (GPIO1): now also R13.2; no longer R14.2
- net at U2.A24 (R1EXT): now also R10.1; no longer R10.2
- net at U2.B23 (R1EXTRTN): now also R10.2; no longer R10.1
- net at R11.2: now also U2.B48 (GPIO3); no longer U2.B47 (GPIO2)
- net at R12.2: now also U2.B47 (GPIO2); no longer U2.B48 (GPIO3)
Other:
- company: 3mdeb Sp. z o.o -> 3mdeb Sp. z o.o    Jakub Sobota
- moved on the sheet: C36, R10, R23, R24, R25, R26, R27, U2

Commit message: Updated PCB Design
Signed-off-by: Jakub Sobota <jakub.sobota@3mdeb.com>
Parts:
- U2: footprint TUSB7320:Texas_tusb7340 -> TUSB7320:Texas_tusb7320
Connections:
- net GND: no longer U2.A53 (PAD)
- net at C35.2, R27.2, U2.A23 (XI): now also Y2.1; no longer Y2.3
- net at C36.2, R27.1, U2.A22 (XO): now also Y2.3; no longer Y2.1
Other:
- moved on the sheet: Y2
Changed lines of the file:
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@@
-	)
-	(junction
-		(at 166.37 160.02)
-		(diameter 0)
-		(color 0 0 0 0)
 	)
 	(junction
@@
 	(wire
 		(pts
-			(xy 166.37 160.02) (xy 166.37 162.56)
-		)
-		(stroke
-			(width 0)
-			(type default)
-		)
-	)
-	(wire
-		(pts
 			(xy 138.43 27.94) (xy 138.43 31.75)
 		)
@@
 	(wire
 		(pts
-			(xy 168.91 158.75) (xy 168.91 160.02)
-		)
-		(stroke
-			(width 0)
-			(type default)
-		)
-	)
-	(wire
-		(pts
 			(xy 229.87 128.27) (xy 236.22 128.27)
 		)
@@
 	(wire
 		(pts
-			(xy 168.91 160.02) (xy 166.37 160.02)
-		)
-		(stroke
-			(width 0)
-			(type default)
-		)
-	)
-	(wire
-		(pts
 			(xy 161.29 27.94) (xy 161.29 31.75)
 		)
@@
 	(wire
 		(pts
-			(xy 166.37 158.75) (xy 166.37 160.02)
+			(xy 166.37 158.75) (xy 166.37 162.56)
 		)
 		(stroke
@@
 	(symbol
 		(lib_id "Device:Crystal_GND24_Small")
-		(at 58.42 67.31 0)
+		(at 58.42 67.31 180)
 		(unit 1)
 		(exclude_from_sim no)
@@
 		(dnp no)
 		(property "Reference" "Y2"
-			(at 55.372 68.834 0)
+			(at 60.96 70.104 0)
 			(effects
 				(font
@@
 		)
 		(property "Value" "48 MHz"
-			(at 63.754 68.834 0)
+			(at 53.594 70.104 0)
 			(effects
 				(font
@@
 			)
 		)
-		(property "Footprint" "TUSB7320:Texas_tusb7340"
+		(property "Footprint" "TUSB7320:Texas_tusb7320"
 			(at 224.79 156.21 0)
 			(effects
@@
 		(pin "A5"
 		)
-		(pin "A53"
-		)
 		(pin "A16"
 		)
@@
 		(pin "A21"
 		)
-		(pin "NC"
-		)
 		(pin "B21"
 		)
@@
 		(pin "B5"
 		)
+		(pin "A8"
+		)
 		(instances

Commit message: Updated 3D models
Signed-off-by: Jakub Sobota <jakub.sobota@3mdeb.com>
Parts:
- renumbered Y2 to Y1
Changed lines of the file:
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@@
 		(on_board yes)
 		(dnp no)
-		(property "Reference" "Y2"
+		(property "Reference" "Y1"
 			(at 60.96 70.104 0)
 			(effects
@@
 			(project ""
 				(path "/513f496d-ec7a-4c1e-814f-35a10c718f03/c66d1eec-955e-444d-af71-f46ce926b72b"
-					(reference "Y2")
+					(reference "Y1")
 					(unit 1)
 				)

Commit message: Cleaned custom libraries, fixed footprint and 3d models
Signed-off-by: Jakub Sobota <jakub.sobota@3mdeb.com>
Parts:
- removed U2: TUSB7320, TUSB7320:Texas_tusb7320, symbol TUSB7320:TUSB7320
- removed Y1: 48 MHz, Crystal:Crystal_SMD_Abracon_ABM3B-4Pin_5.0x3.2mm, symbol Device:Crystal_GND24_Small
- added IC1: TUSB7320RKMT, TUSB7320:TUSB7320RKMT, symbol TUSB7320:TUSB7320RKMT
- added Y1: Crystal, ABM3B:ABM3B-48.000MHZ-B2-T, symbol ABM3B:ABM3B-48.000MHZ-B2-T
- R24, R25: footprint LED_SMD:LED_0402_1005Metric_Pad0.77x0.64mm_HandSolder -> Resistor_SMD:R_0402_1005Metric_Pad0.72x0.64mm_HandSolder
Connections:
- net +1.1V: now also IC1.A1 (VDD11), IC1.A12 (VDD11), IC1.A16 (VDD11), IC1.A28 (VDD11), IC1.A31 (VDD11), IC1.A33 (VDD11), IC1.A38 (VDD11), IC1.A4 (VDD11), IC1.A50 (VDD11), IC1.A6 (VDD11), IC1.A9 (VDD11), IC1.B1 (VDD11), IC1.B17 (VDD11), IC1.B19 (VDD11), IC1.B24 (VDD11), IC1.B37 (VDD11), IC1.B40 (VDD11), IC1.B42 (VDD11), IC1.B44 (VDD11)
- net +3.3V: now also IC1.A3 (VDD33), IC1.A34 (VDD33), IC1.A39 (VDD33), IC1.A47 (VDD33), IC1.A51 (VDD33)
- net DM1: now also IC1.B18 (USB_DM_DN1)
- net DM2: now also IC1.A13 (USB_DM_DN2)
- net DP1: now also IC1.A20 (USB_DP_DN1)
- net DP2: now also IC1.B12 (USB_DP_DN2)
- net GND: now also IC1.B20 (GND), IC1.B32 (JTAG_RST#), Y1.2, Y1.4
- net GRSTZ: now also IC1.A15 (GRST#)
- net OVERCUR1Z: now also IC1.A36 (OVERCUR1#)
- net OVERCUR2Z: now also IC1.A37 (OVERCUR2#)
- net PCIE_REFCLKN: now also IC1.B41 (PCIE_REFCLKN)
- net PCIE_REFCLKP: now also IC1.A45 (PCIE_REFCLKP)
- net PCIE_RXN: now also IC1.A42 (PCIE_RXN)
- net PCIE_RXP: now also IC1.B39 (PCIE_RXP)
- net PCIE_TXN: now also IC1.A41 (PCIE_TXN)
- net PCIE_TXP: now also IC1.B38 (PCIE_TXP)
- net PERSTZ: now also IC1.A40 (PERST#)
- net PWRON1Z: now also IC1.B33 (PWRON1#)
- net PWRON2Z: now also IC1.B34 (PWRON2#)
- net VDDA_3P3: now also IC1.A19 (VDDA_3P3), IC1.A21 (VDDA_3P3), IC1.A25 (VDDA_3P3), IC1.A44 (VDDA_3P3), IC1.B11 (VDDA_3P3), IC1.B22 (VDDA_3P3), IC1.B26 (VDDA_3P3), IC1.B4 (VDDA_3P3)
- net WAKEZ: now also IC1.B35 (WAKE#)
- net at R11.2: now also IC1.B48 (GPIO3)
- net at R12.2: now also IC1.B47 (GPIO2)
- net at R22.1, R23.1: now also IC1.A52 (AUX_DET)
- net at R26.2: now also IC1.B14 (FREQSEL)
- net at C35.1, C36.1: now also IC1.B21 (VSS_OSC)
- net at C35.2, R27.2: now also IC1.A23 (XI), Y1.3
- net at R24.1: now also IC1.A2 (SDA)
- net at C36.2, R27.1: now also IC1.A22 (XO), Y1.1
- net at R14.2: now also IC1.A49 (GPIO0)
- net at R10.1: now also IC1.A24 (R1EXT)
- net at R25.1: now also IC1.B2 (SCL)
- net at R10.2: now also IC1.B23 (R1EXTRTN)
- net at R13.2: now also IC1.B46 (GPIO1)

Commit message: Redesigned PCB compliant with PCI and SS USB standards
Signed-off-by: Jakub Sobota <jakub.sobota@3mdeb.com>
Parts:
- added D8: ESDS304DBVR, ESDS304:ESDS304DBVR, symbol ESDS304DBVR:ESDS304DBVR
- IC1: value TUSB7320RKMT -> TUSB7320
- Y1: value Crystal -> 48 MHz
Connections:
- net DM1: now also D8.5 (I/O4)
- net DM2: now also D8.1 (I/O1)
- net DP1: now also D8.4 (I/O3)
- net DP2: now also D8.3 (I/O2)
- net GND: now also IC1.A53 (GND), D8.2 (GND)

Commit message: fixed pdf schematics, removed temporary files
Signed-off-by: Jakub Sobota <jakub.sobota@3mdeb.com>
Connections:
- net DM1: now also D8.4 (I/O4); no longer D8.5 (I/O4)
- net DP1: now also D8.5 (I/O5); no longer D8.4 (I/O3)
Other:
- moved on the sheet: D8

Commit message: Updated all SMD footprints to not hand soldered versions
Signed-off-by: Jakub Sobota <jakub.sobota@3mdeb.com>
Parts:
- C35, C36: footprint Capacitor_SMD:C_0402_1005Metric_Pad0.74x0.62mm_HandSolder -> Capacitor_SMD:C_0402_1005Metric
- R10, R23, R24, R25, R26, R27: footprint Resistor_SMD:R_0402_1005Metric_Pad0.72x0.64mm_HandSolder -> Resistor_SMD:R_0402_1005Metric
Changed lines of the file:
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@@
 		)
 		(instances
-			(project ""
+			(project "PCI2USB"
 				(path "/513f496d-ec7a-4c1e-814f-35a10c718f03/c66d1eec-955e-444d-af71-f46ce926b72b"
 					(reference "#PWR049")
@@
 			)
 		)
-		(property "Footprint" "Resistor_SMD:R_0402_1005Metric_Pad0.72x0.64mm_HandSolder"
+		(property "Footprint" "Resistor_SMD:R_0402_1005Metric"
 			(at 35.306 124.714 90)
 			(effects
@@
 			)
 		)
-		(property "Footprint" "Resistor_SMD:R_0402_1005Metric_Pad0.72x0.64mm_HandSolder"
+		(property "Footprint" "Resistor_SMD:R_0402_1005Metric"
 			(at 81.534 91.694 90)
 			(effects
@@
 		)
 		(instances
-			(project ""
+			(project "PCI2USB"
 				(path "/513f496d-ec7a-4c1e-814f-35a10c718f03/c66d1eec-955e-444d-af71-f46ce926b72b"
 					(reference "#PWR026")
@@
 			)
 		)
-		(property "Footprint" "Capacitor_SMD:C_0402_1005Metric_Pad0.74x0.62mm_HandSolder"
+		(property "Footprint" "Capacitor_SMD:C_0402_1005Metric"
 			(at 64.77 55.88 0)
 			(effects
@@
 				)
 				(justify right)
-				(hide yes)
-			)
-		)
-		(property "Footprint" "Resistor_SMD:R_0402_1005Metric_Pad0.72x0.64mm_HandSolder"
+			)
+		)
+		(property "Footprint" "Resistor_SMD:R_0402_1005Metric"
 			(at 85.344 108.966 90)
 			(effects
@@
 		)
 		(instances
-			(project ""
+			(project "PCI2USB"
 				(path "/513f496d-ec7a-4c1e-814f-35a10c718f03/c66d1eec-955e-444d-af71-f46ce926b72b"
 					(reference "#PWR038")
@@
 		)
 		(instances
-			(project ""
+			(project "PCI2USB"
 				(path "/513f496d-ec7a-4c1e-814f-35a10c718f03/c66d1eec-955e-444d-af71-f46ce926b72b"
 					(reference "IC1")
@@
 			)
 		)
-		(property "Footprint" "Capacitor_SMD:C_0402_1005Metric_Pad0.74x0.62mm_HandSolder"
+		(property "Footprint" "Capacitor_SMD:C_0402_1005Metric"
 			(at 52.07 55.88 0)
 			(effects
@@
 		)
 		(instances
-			(project ""
+			(project "PCI2USB"
 				(path "/513f496d-ec7a-4c1e-814f-35a10c718f03/c66d1eec-955e-444d-af71-f46ce926b72b"
 					(reference "Y1")
@@
 			)
 		)
-		(property "Footprint" "Resistor_SMD:R_0402_1005Metric_Pad0.72x0.64mm_HandSolder"
+		(property "Footprint" "Resistor_SMD:R_0402_1005Metric"
 			(at 58.674 77.724 90)
 			(effects
@@
 			)
 		)
-		(property "Footprint" "Resistor_SMD:R_0402_1005Metric_Pad0.72x0.64mm_HandSolder"
+		(property "Footprint" "Resistor_SMD:R_0402_1005Metric"
 			(at 63.246 126.746 90)
 			(effects
@@
 				)
 				(justify right)
-				(hide yes)
-			)
-		)
-		(property "Footprint" "Resistor_SMD:R_0402_1005Metric_Pad0.72x0.64mm_HandSolder"
+			)
+		)
+		(property "Footprint" "Resistor_SMD:R_0402_1005Metric"
 			(at 72.644 108.966 90)
 			(effects
