File: Kicad-Files/USBController.kicad_sch (KiCad schematic)
At the start: 16 parts, among them IC1 TUSB7320, Y1 48 MHz

Commit message: Redesigned schematic and board REV 2.0
Parts:
- removed D8: ESDS304DBVR, ESDS304:ESDS304DBVR, symbol ESDS304DBVR:ESDS304DBVR
- removed R11, R12, R13, R14: NOPOP, Resistor_SMD:R_0402_1005Metric_Pad0.72x0.64mm_HandSolder, symbol Device:R_US
- removed R24, R25: 0 Ohm, Resistor_SMD:R_0402_1005Metric, symbol Device:R_US
- removed Y1: 48 MHz, ABM3B:ABM3B-48.000MHZ-B2-T, symbol ABM3B:ABM3B-48.000MHZ-B2-T
- added U2: TPD4EUSB30, Package_SON:USON-10_2.5x1.0mm_P0.5mm, symbol Power_Protection:TPD4EUSB30
- added Y1: 48Mhz, Crystal:Crystal_SMD_3225-4Pin_3.2x2.5mm, symbol Device:Crystal_GND24
- C6: renamed from C35; value 18pF -> 18p
- C7: renamed from C36; value 18pF -> 18p
- R1: renamed from R23; value 10 KOhm -> 10K; now not fitted; now left out of the parts list
- R2: renamed from R22; value NOPOP -> 10K; footprint Resistor_SMD:R_0402_1005Metric_Pad0.72x0.64mm_HandSolder -> Resistor_SMD:R_0402_1005Metric
- R3: renamed from R27; value 1 MOhm -> 1M
- R4: renamed from R10; value 9.09 KOhm -> 9.09K_1%
- R5: renamed from R26; value 4.7 KOhm -> 4.7K
- renumbered IC1 to U1
Connections:
- net GND: now also U1.A2 (SDA), U1.B2 (SCL), U2.3 (GND), U2.8 (GND), Y1.2 (G), Y1.4 (G)
- net OSC_VSS: now reaches C6.1, C7.1, U1.B21 (VSS_OSC)
- net OSC_XO: now reaches C6.2, R3.2
- net OSC_XO: now also U1.A22 (XO), Y1.1; no longer U1.A23 (XI)
- net OSC_XI: now reaches C7.2, R3.1
- net OSC_XI: now also U1.A23 (XI), Y1.3; no longer U1.A22 (XO)
- net CLKREQZ: now reaches U1.B36 (CLKREQ#)
- net DM1 renamed USB_D1N
- net USB_D1N: now also U2.4 (D2+), U2.7 (NC)
- net DM2 renamed USB_D2N
- net USB_D2N: now also U2.2 (D1-), U2.9 (NC)
- net DP1 renamed USB_D1P
- net USB_D1P: now also U2.5 (D2-), U2.6 (NC)
- net DP2 renamed USB_D2P
- net USB_D2P: now also U2.1 (D1+), U2.10 (NC)
- net VDDA_3P3 renamed VDDA
- no-connect marks 0 -> 4
Other:
- company: 3mdeb Sp. z o.o    Jakub Sobota -> 3mdeb Sp. z o.o    Dominik Baroński
- title: PCI2USB -> PCI2USB TUSB7320
- moved on the sheet: C6, C7, R2, R3, R4, R5
